File: Breakouts/Breakouts.brd (EAGLE design)
At the start: 100.4 x 73.3 mm, 41 parts, among them IC1 LD117ADT-TR, IC2 LD117ADT-TR, IC3 4050D, IC4 4050D, IC5 LD117ADT-TR, IC6 4050D, SW1 EC12E_SW, SW2 EC12E_SW, SW3 EC12E_SW, SW4 EC12E_SW, U1 USD-SOCKETUSD, U2 USD-SOCKETUSD, U3 USD-SOCKETUSD

Commit message: Misc updates
Parts:
- added B1, B2: (no value), PatternAgents-TouchWidgets:BUTTON_PASSIVE_10MM
- added B3: (no value), PatternAgents-TouchWidgets:BUTTON_PASSIVE_12MM
- added JP11: M05X2SHD_LOCK, SparkFun-Connectors:2X5-SHROUDED_LOCK
- added SL1: SLIDER_PASSIVE_5SEG, PatternAgents-TouchWidgets:SLIDER_PASSIVE_5SEG_12MM
Connections:
- new net B1: B1.BUTTON, JP11.8
- new net B2: B2.BUTTON, JP11.9
- new net B3: B3.BUTTON, JP11.10
- new net GND6: JP11.1
- new net SL1: JP11.3, SL1.SL1
- new net SL2: JP11.4, SL1.SL2
- new net SL3: JP11.5, SL1.SL3
- new net SL4: JP11.6, SL1.SL4
- new net SL5: JP11.7, SL1.SL5
- new net VCC6: JP11.2
Routing:
- net B2: track 0.00 -> 94.5 mm, vias 0 -> 1
- net B3: track 0.00 -> 73.4 mm
- net B1: track 0.00 -> 58.9 mm, vias 0 -> 1
- net SL5: track 0.00 -> 48.9 mm
- net SL3: track 0.00 -> 36.6 mm
- net SL4: track 0.00 -> 31.6 mm
- net SL2: track 0.00 -> 19.7 mm
- net SL1: track 0.00 -> 19.6 mm
- added copper zone on layer 1, net GND6
- added copper zone on layer 16, net N$14
Other:
- board size 100.4 x 73.3 mm -> 100.4 x 100 mm
- board text added: "SELECT"
Changed lines of the file:
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@@
 <setting verticaltext="up"/>
 </settings>
-<grid distance="0.005125" unitdist="inch" unit="mm" style="lines" multiple="1" display="no" altdistance="0.025" altunitdist="inch" altunit="inch"/>
+<grid distance="0.003125" unitdist="mic" unit="mm" style="lines" multiple="1" display="yes" altdistance="0.025" altunitdist="inch" altunit="inch"/>
 <layers>
 <layer number="1" name="Top" color="4" fill="1" visible="yes" active="yes"/>
@@
 <layer number="223" name="223bmp" color="24" fill="1" visible="no" active="no"/>
 <layer number="224" name="224bmp" color="25" fill="1" visible="no" active="no"/>
+<layer number="231" name="Eagle3D_PG1" color="14" fill="1" visible="yes" active="yes"/>
+<layer number="232" name="Eagle3D_PG2" color="14" fill="2" visible="yes" active="yes"/>
+<layer number="233" name="Eagle3D_PG3" color="14" fill="4" visible="yes" active="yes"/>
 <layer number="248" name="Housing" color="7" fill="1" visible="yes" active="yes"/>
 <layer number="249" name="Edge" color="7" fill="1" visible="yes" active="yes"/>
@@
 <wire x1="-0.390525" y1="0.130175" x2="0" y2="0" width="0.254" layer="20"/>
 <wire x1="0" y1="0" x2="100" y2="0" width="0.254" layer="20"/>
-<wire x1="0" y1="0" x2="0" y2="73.314125" width="0.254" layer="20"/>
-<wire x1="0" y1="73.314125" x2="100" y2="73.314125" width="0.254" layer="20"/>
-<wire x1="100" y1="0" x2="100" y2="73.314125" width="0.254" layer="20"/>
+<wire x1="0" y1="0" x2="0" y2="100" width="0.254" layer="20"/>
+<wire x1="0" y1="100" x2="100" y2="100" width="0.254" layer="20"/>
+<wire x1="100" y1="0" x2="100" y2="100" width="0.254" layer="20"/>
 <text x="8.8519" y="11.585575" size="1.27" layer="255" ratio="17" rot="R90">1k</text>
 <text x="8.8519" y="16.011525" size="1.27" layer="255" ratio="17" rot="R90">1k</text>
@@
 <wire x1="84.8741" y1="50.377725" x2="84.8741" y2="53.37175" width="0.254" layer="255"/>
 <wire x1="84.8741" y1="55.324375" x2="84.8741" y2="58.188225" width="0.254" layer="255"/>
+<rectangle x1="33" y1="81" x2="39" y2="90" layer="255"/>
+<rectangle x1="41" y1="81" x2="47" y2="94" layer="255"/>
+<rectangle x1="25" y1="81" x2="31" y2="87" layer="255"/>
+<rectangle x1="18" y1="81" x2="23" y2="84" layer="255"/>
+<circle x="74.932378125" y="88.752265625" radius="6.6396625" width="0.8128" layer="255"/>
+<circle x="91.4387125" y="87.474253125" radius="5.82020625" width="0.8128" layer="255"/>
+<circle x="58.432625" y="87.481121875" radius="5.7924875" width="0.8128" layer="255"/>
+<wire x1="58.5159125" y1="89.225953125" x2="56.5159125" y2="87.225953125" width="0.8128" layer="255"/>
+<wire x1="58.5159125" y1="89.225953125" x2="60.5159125" y2="87.225953125" width="0.8128" layer="255"/>
+<wire x1="58.5159125" y1="87.225953125" x2="56.5159125" y2="85.225953125" width="0.8128" layer="255"/>
+<wire x1="58.5159125" y1="87.225953125" x2="60.5159125" y2="85.225953125" width="0.8128" layer="255"/>
+<wire x1="91.527078125" y1="85.612975" x2="89.527078125" y2="87.612975" width="0.8128" layer="255"/>
+<wire x1="91.527078125" y1="85.612975" x2="93.527078125" y2="87.612975" width="0.8128" layer="255"/>
+<wire x1="89.527078125" y1="89.612975" x2="91.527078125" y2="87.612975" width="0.8128" layer="255"/>
+<wire x1="91.527078125" y1="87.612975" x2="93.527078125" y2="89.612975" width="0.8128" layer="255"/>
+<text x="69.2513125" y="87.595271875" size="2.1844" layer="255" font="vector" ratio="20">SELECT</text>
 </plain>
 <attributes>
@@
 <attribute name="OC_FARNELL" value="1520813" x="66.843275" y="21.370925" size="1.778" layer="27" rot="R270" display="off"/>
 </element>
+<element name="SL1" library="PatternAgents-TouchWidgets" package="SLIDER_PASSIVE_5SEG_12MM" value="SLIDER_PASSIVE_5SEG" x="33.02" y="87.48395" rot="R270"/>
+<element name="B1" library="PatternAgents-TouchWidgets" package="BUTTON_PASSIVE_10MM" value="" x="58.42" y="87.48395"/>
+<element name="B2" library="PatternAgents-TouchWidgets" package="BUTTON_PASSIVE_10MM" value="" x="91.44" y="87.48395"/>
+<element name="JP11" library="SparkFun-Connectors" package="2X5-SHROUDED_LOCK" value="M05X2SHD_LOCK" x="5" y="88.32395"/>
+<element name="B3" library="PatternAgents-TouchWidgets" package="BUTTON_PASSIVE_12MM" value="" x="74.93" y="88.75395"/>
 </elements>
 <signals>
@@
 <wire x1="82.773275" y1="51.850925" x2="85.273275" y2="54.350925" width="0.6096" layer="16"/>
 </signal>
+<signal name="GND6">
+<contactref element="JP11" pad="1"/>
+<polygon width="0.254" layer="1" pour="hatch" isolate="0.3048">
+<vertex x="0" y="98.91395"/>
+<vertex x="99.06" y="98.91395"/>
+<vertex x="99.06" y="77.32395"/>
+<vertex x="0" y="77.32395"/>
+</polygon>
+</signal>
+<signal name="VCC6">
+<contactref element="JP11" pad="2"/>
+</signal>
+<signal name="B3">
+<contactref element="JP11" pad="10"/>
+<contactref element="B3" pad="BUTTON"/>
+<wire x1="13.208" y1="90.02395" x2="6.604" y2="83.41995" width="0.254" layer="16"/>
+<wire x1="36.576" y1="90.02395" x2="13.208" y2="90.02395" width="0.254" layer="16"/>
+<wire x1="40.894" y1="94.34195" x2="36.576" y2="90.02395" width="0.254" layer="16"/>
+<wire x1="73.914" y1="94.34195" x2="40.894" y2="94.34195" width="0.254" layer="16"/>
+<wire x1="74.676" y1="93.57995" x2="73.914" y2="94.34195" width="0.254" layer="16"/>
+<wire x1="74.93" y1="93.57995" x2="74.676" y2="93.57995" width="0.254" layer="16"/>
+<wire x1="6.604" y1="83.41995" x2="6.397" y2="83.24395" width="0.254" layer="16"/>
+</signal>
+<signal name="SL5">
+<contactref element="SL1" pad="SL5"/>
+<contactref element="JP11" pad="7"/>
+<wire x1="1.778" y1="83.92795" x2="3.556" y2="85.70595" width="0.254" layer="16"/>
+<wire x1="1.778" y1="82.65795" x2="1.778" y2="83.92795" width="0.254" layer="16"/>
+<wire x1="3.048" y1="81.38795" x2="1.778" y2="82.65795" width="0.254" layer="16"/>
+<wire x1="29.464" y1="81.38795" x2="3.048" y2="81.38795" width="0.254" layer="16"/>
+<wire x1="41.148" y1="93.07195" x2="29.464" y2="81.38795" width="0.254" layer="16"/>
+<wire x1="41.402" y1="93.07195" x2="41.148" y2="93.07195" width="0.254" layer="16"/>
+<wire x1="3.556" y1="85.70595" x2="3.603" y2="85.78395" width="0.254" layer="16"/>
+</signal>
+<signal name="SL4">
+<contactref element="SL1" pad="SL4"/>
+<contactref element="JP11" pad="6"/>
+<wire x1="8.636" y1="90.53195" x2="6.604" y2="88.49995" width="0.254" layer="16"/>
+<wire x1="33.274" y1="90.53195" x2="8.636" y2="90.53195" width="0.254" layer="16"/>
+<wire x1="35.814" y1="93.07195" x2="33.274" y2="90.53195" width="0.254" layer="16"/>
+<wire x1="36.068" y1="93.07195" x2="35.814" y2="93.07195" width="0.254" layer="16"/>
+<wire x1="6.604" y1="88.49995" x2="6.397" y2="88.32395" width="0.254" layer="16"/>
+</signal>
+<signal name="SL3">
+<contactref element="SL1" pad="SL3"/>
+<contactref element="JP11" pad="5"/>
+<wire x1="1.778" y1="90.27795" x2="3.556" y2="88.49995" width="0.254" layer="16"/>
+<wire x1="1.778" y1="93.57995" x2="1.778" y2="90.27795" width="0.254" layer="16"/>
+<wire x1="3.81" y1="95.61195" x2="1.778" y2="93.57995" width="0.254" layer="16"/>
+<wire x1="27.686" y1="95.61195" x2="3.81" y2="95.61195" width="0.254" layer="16"/>
+<wire x1="30.226" y1="93.07195" x2="27.686" y2="95.61195" width="0.254" layer="16"/>
+<wire x1="30.48" y1="93.07195" x2="30.226" y2="93.07195" width="0.254" layer="16"/>
+<wire x1="3.556" y1="88.49995" x2="3.603" y2="88.32395" width="0.254" layer="16"/>
+</signal>
+<signal name="SL2">
+<contactref element="SL1" pad="SL2"/>
+<contactref element="JP11" pad="4"/>
+<wire x1="22.86" y1="91.03995" x2="6.604" y2="91.03995" width="0.254" layer="16"/>
+<wire x1="24.892" y1="93.07195" x2="22.86" y2="91.03995" width="0.254" layer="16"/>
+<wire x1="25.146" y1="93.07195" x2="24.892" y2="93.07195" width="0.254" layer="16"/>
+<wire x1="6.604" y1="91.03995" x2="6.397" y2="90.86395" width="0.254" layer="16"/>
+</signal>
+<signal name="SL1">
+<contactref element="SL1" pad="SL1"/>
+<contactref element="JP11" pad="3"/>
+<wire x1="5.08" y1="92.30995" x2="3.81" y2="91.03995" width="0.254" layer="16"/>
+<wire x1="5.08" y1="94.08795" x2="5.08" y2="92.30995" width="0.254" layer="16"/>
+<wire x1="6.096" y1="95.10395" x2="5.08" y2="94.08795" width="0.254" layer="16"/>
+<wire x1="17.272" y1="95.10395" x2="6.096" y2="95.10395" width="0.254" layer="16"/>
+<wire x1="19.304" y1="93.07195" x2="17.272" y2="95.10395" width="0.254" layer="16"/>
+<wire x1="19.558" y1="93.07195" x2="19.304" y2="93.07195" width="0.254" layer="16"/>
+<wire x1="3.81" y1="91.03995" x2="3.603" y2="90.86395" width="0.254" layer="16"/>
+</signal>
+<signal name="B1">
+<contactref element="B1" pad="BUTTON"/>
+<contactref element="JP11" pad="8"/>
+<wire x1="11.938" y1="80.37195" x2="6.604" y2="85.70595" width="0.254" layer="1"/>
+<wire x1="46.99" y1="80.37195" x2="11.938" y2="80.37195" width="0.254" layer="16"/>
+<wire x1="58.166" y1="91.54795" x2="46.99" y2="80.37195" width="0.254" layer="16"/>
+<wire x1="58.42" y1="91.54795" x2="58.166" y2="91.54795" width="0.254" layer="16"/>
+<wire x1="6.604" y1="85.70595" x2="6.397" y2="85.78395" width="0.254" layer="1"/>
+<via x="11.938" y="80.37195" extent="1-16" drill="0.6096"/>
+</signal>
+<signal name="B2">
+<contactref element="B2" pad="BUTTON"/>
+<contactref element="JP11" pad="9"/>
+<wire x1="7.62" y1="79.35595" x2="3.81" y2="83.16595" width="0.254" layer="1"/>
+<wire x1="78.994" y1="79.35595" x2="7.62" y2="79.35595" width="0.254" layer="16"/>
+<wire x1="91.186" y1="91.54795" x2="78.994" y2="79.35595" width="0.254" layer="16"/>
+<wire x1="91.44" y1="91.54795" x2="91.186" y2="91.54795" width="0.254" layer="16"/>
+<wire x1="3.81" y1="83.16595" x2="3.603" y2="83.24395" width="0.254" layer="1"/>
+<via x="7.62" y="79.35595" extent="1-16" drill="0.6096"/>
+</signal>
+<signal name="N$14">
+<polygon width="0.254" layer="16" spacing="1.778" pour="hatch" isolate="0.3048">
+<vertex x="0" y="100.18395"/>
+<vertex x="100.33" y="100.18395"/>
+<vertex x="100.33" y="77.32395"/>
+<vertex x="0" y="77.32395"/>
+</polygon>
+</signal>
 </signals>
