File: Hy28B LCD Board/HY28B-LCD.sch (EAGLE design)
At the start: 32 parts, among them K2 PIN20X2, U2 EEPROM24, X1 RASPI_BOARD_B+_F

Commit message: HY28 and Ramps1.5
Connections:
- net GPIO25: now also K2.22
- net GPIO28: no longer K2.22
Changed lines of the file:
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@@
 <pinref part="X1" gate="G$1" pin="N.C.1"/>
 <wire x1="154.94" y1="48.26" x2="157.48" y2="48.26" width="0.1524" layer="91"/>
+<label x="157.48" y="48.26" size="1.778" layer="95"/>
 </segment>
 <segment>
@@
 </net>
 <net name="GPIO28" class="0">
-<segment>
-<pinref part="K2" gate="G$1" pin="22"/>
-<wire x1="226.06" y1="43.18" x2="228.6" y2="43.18" width="0.1524" layer="91"/>
-<label x="233.68" y="43.18" size="1.778" layer="95"/>
-</segment>
 <segment>
 <pinref part="U$1" gate="G$1" pin="RST"/>
@@
 <pinref part="X1" gate="G$1" pin="N.C.8"/>
 <wire x1="154.94" y1="30.48" x2="157.48" y2="30.48" width="0.1524" layer="91"/>
+<label x="157.48" y="30.48" size="1.778" layer="95"/>
 </segment>
 </net>
@@
 <pinref part="X1" gate="G$1" pin="N.C.7"/>
 <wire x1="154.94" y1="33.02" x2="157.48" y2="33.02" width="0.1524" layer="91"/>
+<label x="157.48" y="33.02" size="1.778" layer="95"/>
 </segment>
 </net>
@@
 <pinref part="X1" gate="G$1" pin="N.C.6"/>
 <wire x1="154.94" y1="35.56" x2="157.48" y2="35.56" width="0.1524" layer="91"/>
+<label x="157.48" y="35.56" size="1.778" layer="95"/>
 </segment>
 </net>
@@
 <pinref part="X1" gate="G$1" pin="N.C.5"/>
 <wire x1="154.94" y1="38.1" x2="157.48" y2="38.1" width="0.1524" layer="91"/>
+<label x="157.48" y="38.1" size="1.778" layer="95"/>
 </segment>
 </net>
@@
 <pinref part="X1" gate="G$1" pin="N.C.4"/>
 <wire x1="154.94" y1="40.64" x2="157.48" y2="40.64" width="0.1524" layer="91"/>
+<label x="157.48" y="40.64" size="1.778" layer="95"/>
 </segment>
 </net>
@@
 <pinref part="X1" gate="G$1" pin="N.C.3"/>
 <wire x1="154.94" y1="43.18" x2="157.48" y2="43.18" width="0.1524" layer="91"/>
+<label x="157.48" y="43.18" size="1.778" layer="95"/>
 </segment>
 </net>
@@
 <pinref part="X1" gate="G$1" pin="N.C.2"/>
 <wire x1="154.94" y1="45.72" x2="157.48" y2="45.72" width="0.1524" layer="91"/>
+<label x="157.48" y="45.72" size="1.778" layer="95"/>
 </segment>
 </net>
@@
 <label x="111.76" y="50.8" size="1.778" layer="95"/>
 </segment>
-</net>
+<segment>
+<pinref part="K2" gate="G$1" pin="22"/>
+<wire x1="226.06" y1="43.18" x2="228.6" y2="43.18" width="0.1524" layer="91"/>
+<label x="233.68" y="43.18" size="1.778" layer="95"/>
+</segment>
+</net>
