File: OpenHardware.co.za Controller V3.6/TestBench_rev3.6.brd (EAGLE design)
At the start: 100 x 100 mm, 100 parts, among them IC1 MCP2200SOIC20, IC2 ATMEGA644-20PU, IC3 7805TV, IC4 LD117ADT-TR, IC7 4050D, Q1 12Mhz, Q7 20Mhz, SW1 SPST_TACT-EVQQ2, U1 USD-SOCKETUSD, X1 USBPTH

Commit message: HY28 and Ramps1.5
Parts:
- removed BED, VMOT: (no value), con-wago-500:W237-102
- removed D6: (no value), SparkFun-DiscreteSemi:SMA-DIODE_ALT
- removed E1: E1, SparkFun-Connectors:SCREWTERMINAL-3.5MM-2
- removed E2: E2, SparkFun-Connectors:SCREWTERMINAL-3.5MM-2
- removed E2POL: POLOLU_A4983CARRIER, RepRapjr:A4988BREAKOUT
- removed FAN1: FAN, SparkFun-Connectors:SCREWTERMINAL-3.5MM-2
- removed JP1: (no value), jumper:JP2
- removed JP2: (no value), SparkFun-Connectors:SCREWTERMINAL-3.5MM-4
- removed JP4: (no value), SparkFun-Connectors:SCREWTERMINAL-3.5MM-2
- removed JP6: M05X2SHD_LOCK, SparkFun-Connectors:2X5-SHROUDED_LOCK
- removed PWRLED1, SCKLED1: (no value), LilyPad-Wearables:LED-1206
- removed Q1: 12Mhz, adafruit:HC49UP
- removed Q3, Q4, Q5, Q6: (no value), transistor-power:TO220BV
- removed R12: 4k7, resistor:M1206
- removed R13, R18, R21: 10R, resistor:M1206
- removed R14: (no value), adafruit:M1206
- removed R17: (no value), SparkFun-Passives:1206
- removed R3: 1k, resistor:M1206
- removed TXLED, TXLED1, VCCOK: (no value), led:1206
- removed X1: USBPTH, SparkFun-Connectors:USB-B-PTH
- added 12MHZ1: (no value), crystal:HC49UP
- added JP10: (no value), pinhead:2X03/90
- added LED1, LED2: (no value), adafruit:1206
- added U$2: CH340G, usb-serial:SOIC16
- added U$3, U$4: IRLR8743, IRLR8743:TO263
- added U$5: XY825A-8P, Communica.co.za:XY825A-8P
- added X2: (no value), con-berg:PN61729
- C1, C2: value 22 -> 10u; device SparkFun-Passives:1206 -> rcl:SANYO-OSCON_SMD_B6
- C16, C17: value (none) -> 22
- C21: value 10u -> 0.1u; device rcl:SANYO-OSCON_SMD_B6 -> SparkFun-Passives:1206
- C3, C4: value 0.1u -> 10u; device SparkFun-Passives:1206 -> rcl:SANYO-OSCON_SMD_B6
- IC1: value MCP2200SOIC20 -> 4050D; device microchip-update-2:SOIC20 -> 40xx:SO16
- JP18, JP19, JP20, JP5, JP7: value (none) -> M023.5MM
- R1: value 10k -> 10R
- R2: value 1k -> 10R
- U$1: value LABEL_JUMPER_1X3 -> IRLR8743; device dp_devices:JUMP3_DESC -> IRLR8743:TO263
- moved U1 322.4 mm to (145.4, 49.2), turned to 90 degrees
- moved R9 321.6 mm to (134.6, 55.2), turned to 90 degrees
- moved IC7 318.0 mm to (133.7, 45.1)
- moved C27 314.5 mm to (131.4, 75.9), turned to 90 degrees
- moved C28 310.3 mm to (127.3, 55.2), turned to 270 degrees
- moved JP18 308.1 mm to (173.2, -64.7), turned to 180 degrees
- moved IC4 306.2 mm to (125.7, 65.7), turned to 180 degrees
- moved ZENDSTOP2 302.9 mm to (170.7, -61.8), turned to 0 degrees
- moved JP19 302.6 mm to (164.3, -64.7), turned to 180 degrees
- moved JP20 297.5 mm to (155.4, -64.7), turned to 180 degrees
- moved YENDSTOP2 297.4 mm to (161.8, -61.8), turned to 0 degrees
- moved XENDSTOP2 292.3 mm to (152.9, -61.8), turned to 0 degrees
- moved SW1 271.2 mm to (150.8, 19.4), turned to 270 degrees
- moved R4 262.6 mm to (142.6, 30.8), turned to 180 degrees
- moved R20 251.0 mm to (122.9, -48.3)
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Connections:
- removed net 5VREG: C30.+, IC3.3, JP1.1
- removed net BEDOUT1: BED.1, D6.A, Q3.D
- removed net BEDOUT2: D3.A, E1.2, Q5.D
- removed net DO: U1.7
- removed net E1OUT1: D2.A, E2.2, Q4.D
- removed net E2MSFT: IC2.19, R18.1
- removed net E2STEP: E2POL.STEP, IC2.26
- removed net EXT2ADC: C21.+, IC2.33, JP4.2, R12.2
- removed net FANOUT1: D1.A, FAN1.2, Q6.D
- removed net N$10: R3.1, TXLED1.C
- removed net N$13: IC1.4, R1.1
- removed net N$42: E2POL.1B, JP2.4
- removed net N$43: E2POL.1A, JP2.3
- removed net N$44: E2POL.2A, JP2.2
- removed net N$45: E2POL.2B, JP2.1
- removed net N$49: PWRLED1.A, R14.2
- removed net N$55: Q6.G, R13.2
- removed net N$61: Q4.G, R18.2
- removed net N$67: Q3.G, R21.2
- removed net N$73: JP6.8
- removed net N$9: R2.1, TXLED.C
- removed net VUSB: C4.1, IC1.1, JP1.3, R1.2, TXLED.A, TXLED1.A, X1.VBUS
- new net BEDOUT: D1.A, U$3.3, U$5.3
- new net D+: U$2.5, X2.3
- new net D-: U$2.6, X2.2
- new net EXTOUT: D3.A, U$1.3, U$5.5
- new net FANOUT: D2.A, U$4.3, U$5.7
- new net N$38: 12MHZ1.1, C16.1, U$2.7
- new net N$40: 12MHZ1.2, C17.1, U$2.8
- net 5V: now also U$2.16, X2.1; no longer C27.2, IC4.3
- net BEDMSFT: now also R1.1; no longer R21.1
- net E1DIR: no longer E2POL.DIR
- net ENABLE: no longer E2POL.EN
- net FANMSFT: now also R2.1; no longer R13.1
- net GND: now also C1.-, C16.2, C2.-, C21.2, C3.-, C4.-, IC1.8, JP10.6, LED1.C, LED2.C, U$1.2, U$2.1, U$3.2, U$4.2, U$5.1, X2.4; no longer C1.2, C16.1, C2.1, C21.-, C3.1, C4.2, E2POL.GND, E2POL.GND@0, IC1.20, JP4.1, JP6.6, PWRLED1.C, Q3.S, Q4.S, Q5.S, Q6.S, SCKLED1.C, VCCOK.C, VMOT.1, X1.GND
- net MCRTS: now also U$2.13; no longer IC1.11
- net MCRX: now also U$2.3; no longer IC1.12
- net MCTX: now also U$2.2; no longer IC1.10
- net MCURESET: now also JP10.5; no longer JP6.5
- net MISO: now also JP10.1, U1.7; no longer JP6.1
- net MOSI: now also JP10.4; no longer JP6.4
- net N$1: now also IC1.5; no longer C2.2, IC1.2, Q1.1
- net N$2: no longer C1.1, Q1.2
- net N$3: now also IC1.2; no longer IC1.5, R2.2
- net N$39: now also LED2.A; no longer SCKLED1.A
- net N$4: now also IC1.7; no longer IC1.18, X1.D-
- net N$41: now also C21.1, U$2.4; no longer E2POL.MS1, E2POL.MS2, E2POL.MS3, R17.2
- net N$46: now also U$1.1; no longer Q5.G
- net N$5: now also IC1.6; no longer IC1.19, X1.D+
- net N$6: now also IC1.4; no longer IC1.6, R3.2
- net N$64: now also LED1.A; no longer VCCOK.A
- net N$7: now also R1.2, U$3.1; no longer C3.2, IC1.17
- net N$8: now also R2.2, U$4.1; no longer E2POL.RST, E2POL.SLP
- net SCK: now also JP10.3; no longer JP6.3
- net SCL: no longer JP6.10
- net SDA: no longer JP6.9
- net SDS: no longer JP6.7
- net VCC: now also C27.2, C30.+, IC1.1, IC3.3, IC4.3, JP10.2; no longer C17.1, E2POL.VDD, JP1.2, JP6.2, R12.1, R14.1, R17.1
- net VMOT: now also C1.+, C2.+, C3.+, C4.+, U$5.2, U$5.4, U$5.6, U$5.8; no longer BED.2, C16.2, D6.C, E1.1, E2.1, E2POL.VMOT, FAN1.1, VMOT.2
Routing:
- net GND: track 647.1 -> 411.7 mm, vias 3 -> 6
- net ENABLE: track 235.9 -> 88.3 mm
- net VMOT: track 257.6 -> 116.1 mm, vias 3 -> 0
- net BEDADC: track 116.2 -> 0.00 mm, vias 3 -> 0
- net VCC: track 400.0 -> 287.4 mm, vias 13 -> 4
- net EXTADC: track 89.4 -> 0.00 mm, vias 3 -> 0
- net SCL: track 70.5 -> 0.00 mm
- net BEDMSFT: track 67.3 -> 0.00 mm, vias 2 -> 0
- net VUSB: track 64.2 -> 0.00 mm, vias 1 -> 0
- net EXT2ADC: track 62.9 -> 0.00 mm, vias 2 -> 0
- net SDA: track 60.4 -> 0.00 mm
- net 3V3SD: track 0.00 -> 58.7 mm, vias 0 -> 3
- net E1DIR: track 64.9 -> 11.3 mm, vias 3 -> 0
- net E2MSFT: track 50.9 -> 0.00 mm, vias 1 -> 0
- net EXTMSFT: track 43.2 -> 0.00 mm
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- removed copper zone on layer 1, net 5V
- removed copper zone on layer 16, net GND
- removed copper zone on layer 1, net VCC
- removed copper zone on layer 1, net VMOT
Other:
- board text removed: "+"
- board text removed: "-"
- board text removed: "- +"
- board text removed: ".CO.ZA"
- board text removed: "0.1u"
- board text removed: "1"
- board text removed: "100uF"
- board text removed: "10K"
- board text removed: "10R"
- board text removed: "10uF"
- board text removed: "10uH"
- board text removed: "12Mhz"
- board text removed: "12V 15A IN"
- board text removed: "12V IN"
- board text removed: "1B"
- board text removed: "1K"
- board text removed: "20Mhz"
- board text removed: "22p"
- board text removed: "2B"
- board text removed: "4K7"
- board text removed: "5V"
- board text removed: "5V SOURCE"
- board text removed: "7805"
- board text removed: "ATMEGA1284P"
- board text removed: "BUZZER"
- board text removed: "Bed"
- board text removed: "CC-BY-NC"
- board text removed: "D1"
- board text removed: "D2"
- board text removed: "D3"
- board text removed: "D4"
- board text removed: "DIR"
- board text removed: "E1"
- board text removed: "E1MOTOR"
- board text removed: "E2"
- board text removed: "E2MOTOR"
- board text removed: "EN"
- board text removed: "ENA"
- board text removed: "ENB"
- board text removed: "ENC"
- board text removed: "Endstops:"
- board text removed: "Extruder"
- board text removed: "Extruder 1"
- board text removed: "Extruder 2"
- board text removed: "Extruder Fan"
- board text removed: "FAN"
- board text removed: "GND"
- board text removed: "H/E1"
- board text removed: "H/E2"
- board text removed: "HARDWARE"
- board text removed: "HEATBED"
- board text removed: "Heatbed"
- board text removed: "Heater"
- board text removed: "Hotend"
- board text removed: "Hotend 2"
- board text removed: "IRBL8743"
- board text removed: "IRFZ44N"
- board text removed: "LCD/SD"
- board text removed: "LEDS"
- board text removed: "M1"
- board text removed: "M2"
- board text removed: "M3"
- board text removed: "MCP2200"
- board text removed: "MISO"
- board text removed: "MOSI"
- board text removed: "OPEN"
- board text removed: "Optional"
- board text removed: "POWER"
- board text removed: "Peter vd Walt (2014)"
- board text removed: "RESET"
- board text removed: "RST"
- board text removed: "RX"
- board text removed: "SCK"
- board text removed: "SCL"
- board text removed: "SDA"
- board text removed: "SDS(14)"
- board text removed: "SIG"
- board text removed: "SIG=NO on Switch GND=C on Switch"
- board text removed: "SLP"
- board text removed: "STEP"
- board text removed: "Single"
- board text removed: "Stepper Motor"
- board text removed: "Stepper Motor Wiring 1=BLACK 2=GREEN 3=BLUE 4=RED"
- board text removed: "TX"
- board text removed: "Therm"
- board text removed: "Thermistor"
- board text removed: "USB"
- board text removed: "V3.51.1-BBT"
- board text removed: "WWW."
- board text removed: "X"
- board text removed: "X-MIN"
- board text removed: "X-MOTOR"
- board text removed: "XMOTOR"
- board text removed: "Y"
- board text removed: "Y-MIN"
- board text removed: "Y-MOTOR"
- board text removed: "YMOTOR"
- board text removed: "Z"
- board text removed: "Z-MIN"
- board text removed: "Z-MOTOR"
- board text removed: "Z:/Logos/logo.bmp"
- board text removed: "ZMOTOR"

Commit message: V3.6 with GooglePlus Interconnect Ideas
Parts:
- removed JP10: (no value), pinhead:2X03/90
- removed JP12, JP13, JP14, JP17: (no value), SparkFun-Connectors:SCREWTERMINAL-3.5MM-4
- removed JP18, JP19, JP20: M023.5MM, SparkFun-Connectors:SCREWTERMINAL-3.5MM-2
- removed PCB1: PCB_DP_SQUARE-10X10, dp_devices:DP100100_V1
- removed SG1: F/CM12P, buzzer:F/CM12P
- removed XENDSTOP2, YENDSTOP2, ZENDSTOP2: 22-23-2031, con-molex:22-23-2031
- added BUZZER: F/CM12P, buzzer:F/CM12P
- added C24, C26, C29: 220u, rcl:153CLV-0605
- added D4, D7: (no value), dp_devices:DO-214AC
- added IC5: (no value), linear:TO263-5
- added JP1: (no value), SparkFun-Connectors:1X04_LOCK
- added JP2, JP4, JP6, JP8: M05X2SHD, SparkFun-Connectors:2X5-SHROUDED
- added L2, L3: 33uH, SparkFun-Passives:CDRH125
- added U$12: M08X2, SparkFun-Connectors:2X8
- added U$6: CQ-121, Mantech.co.za:CQ121
- added U$7: AVR-ISP-6-EDGE, atmega-atxmega:6PAD_ISP
- C25: value 100u -> 220u; device adafruit:PANASONIC_C -> rcl:153CLV-0605
- IC3: value 7805TV -> (none); device linear:TO220V -> linear:TO263-5
- R9: value (none) -> 1K
- moved X2 212.6 mm to (-48.3, 143.8), turned to 270 degrees
- moved C17 207.9 mm to (-45.1, 151.4), turned to 0 degrees
- moved LED2 198.9 mm to (-41.6, 106.4), turned to 180 degrees
- moved U1 195.4 mm to (-38.7, 114.6), turned to 270 degrees
- moved IC1 195.1 mm to (-29.8, -38.5), turned to 270 degrees
- moved 12MHZ1 192.7 mm to (-34.3, 151.4), turned to 180 degrees
- moved C21 190.2 mm to (-39.7, 133.7), turned to 180 degrees
- moved JP5 187.1 mm to (-53.7, 93.0), turned to 270 degrees
- moved U$2 187.0 mm to (-35.6, 141.3), turned to 90 degrees
- moved C7 184.9 mm to (-29.5, 134.0), turned to 180 degrees
- moved R16 183.3 mm to (241.9, -90.8), turned to 0 degrees
- moved C16 182.1 mm to (-22.5, 151.1), turned to 180 degrees
- moved IC7 179.0 mm to (-31.1, 114.9), turned to 90 degrees
- moved R10 178.5 mm to (-47.6, 92.4), turned to 270 degrees
- moved R9 177.1 mm to (-34.9, 106.4), turned to 180 degrees
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Connections:
- removed net N$2: IC1.3
- removed net N$22: E1POL.1B, JP17.4
- removed net N$23: E1POL.1A, JP17.3
- removed net N$24: E1POL.2A, JP17.2
- removed net N$25: E1POL.2B, JP17.1
- removed net N$26: JP14.4, ZPOL.1B
- removed net N$27: JP14.3, ZPOL.1A
- removed net N$28: JP14.2, ZPOL.2A
- removed net N$29: JP14.1, ZPOL.2B
- removed net N$3: IC1.2
- removed net N$30: JP13.1, YPOL.2B
- removed net N$31: JP13.2, YPOL.2A
- removed net N$32: JP13.3, YPOL.1A
- removed net N$33: JP13.4, YPOL.1B
- removed net N$34: JP12.4, XPOL.1B
- removed net N$35: JP12.3, XPOL.1A
- removed net N$36: JP12.2, XPOL.2A
- removed net N$37: JP12.1, XPOL.2B
- removed net N$4: IC1.7
- removed net N$5: IC1.6
- removed net N$6: IC1.4
- new net 12V: C29.+, IC3.4, JP2.9, JP4.9, JP6.9, JP8.9, L3.2, U$12.15
- new net E1A: E1POL.1A, JP8.3
- new net E1B: E1POL.1B, JP8.4
- new net E2A: E1POL.2A, JP8.2
- new net E2B: E1POL.2B, JP8.1
- new net HEATER+: U$12.5, U$12.6, U$12.7, U$12.8
- new net HEATER-: U$12.10, U$12.11, U$12.12, U$12.9
- new net N$9: D7.1, IC5.2, L2.1
- new net PWRIN: U$5.2, U$6.1@1, U$6.2@1
- new net THERMISTOR+: U$12.1, U$12.2
- new net THERMISTOR-: U$12.3, U$12.4
- new net X1A: JP4.3, XPOL.1A
- new net X1B: JP4.4, XPOL.1B
- new net X2A: JP4.2, XPOL.2A
- new net X2B: JP4.1, XPOL.2B
- new net XEND12: IC1.7, JP4.10
- new net Y1A: JP2.3, YPOL.1A
- new net Y1B: JP2.4, YPOL.1B
- new net Y2A: JP2.2, YPOL.2A
- new net Y2B: JP2.1, YPOL.2B
- new net YEND12: IC1.5, JP2.10
- new net Z1A: JP6.3, ZPOL.1A
- new net Z1B: JP6.4, ZPOL.1B
- new net Z2A: JP6.2, ZPOL.2A
- new net Z2B: JP6.1, ZPOL.2B
- new net ZEND12: IC1.3, JP6.10, JP8.10, U$12.16
- net BUZZER: now also BUZZER.+; no longer SG1.+
- net GND: now also BUZZER.-, C24.-, C26.-, C29.-, D4.2, D7.2, IC3.3, IC3.5, IC3.6, IC5.3, IC5.5, IC5.6, JP1.4, JP2.5, JP2.6, JP2.8, JP4.5, JP4.6, JP4.8, JP6.5, JP6.6, JP6.8, JP8.5, JP8.6, JP8.8, U$12.14, U$7.GND; no longer IC3.2, JP10.6, JP18.2, JP19.2, JP20.2, SG1.-, XENDSTOP2.2, YENDSTOP2.2, ZENDSTOP2.2
- net MCURESET: now also U$7.RST; no longer JP10.5
- net MISO: now also U$7.MISO; no longer JP10.1
- net MOSI: now also U$7.MOSI; no longer JP10.4
- net N$1: now also D4.1, IC3.2, L3.1; no longer IC1.5
- net SCK: now also U$7.SCK; no longer JP10.3
- net SCL: now also JP1.1
- net SDA: now also JP1.2
- net VCC: now also C26.+, IC5.4, JP1.3, JP2.7, JP4.7, JP6.7, JP8.7, L2.2, U$12.13, U$7.VCC; no longer IC3.3, JP10.2, XENDSTOP2.1, YENDSTOP2.1, ZENDSTOP2.1
- net VMOT: now also C24.+, IC5.1, U$6.3@2, U$6.4@2; no longer U$5.2
- net XEND: now also IC1.6; no longer JP20.1, XENDSTOP2.3
- net YEND: now also IC1.4; no longer JP19.1, YENDSTOP2.3
- net ZEND: now also IC1.2; no longer JP18.1, ZENDSTOP2.3
Routing:
- net GND: track 411.7 -> 0.00 mm, vias 6 -> 0
- net VCC: track 287.4 -> 0.00 mm, vias 4 -> 0
- net VMOT: track 116.1 -> 0.00 mm
- net ENABLE: track 88.3 -> 0.00 mm, vias 1 -> 0
- net MCURESET: track 87.0 -> 0.00 mm, vias 2 -> 0
- net MCRX: track 61.6 -> 0.00 mm
- net MCTX: track 59.4 -> 0.00 mm
- net 3V3SD: track 58.7 -> 0.00 mm, vias 3 -> 0
- net SDS: track 57.3 -> 0.00 mm, vias 1 -> 0
- net MOSI: track 57.0 -> 0.00 mm, vias 3 -> 0
- net SCK: track 55.3 -> 0.00 mm, vias 2 -> 0
- net MISO: track 53.7 -> 0.00 mm, vias 1 -> 0
- net AVCC: track 46.0 -> 0.00 mm, vias 1 -> 0
- net MCRTS: track 43.1 -> 0.00 mm, vias 2 -> 0
- net ENCC: track 29.7 -> 0.00 mm
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- added copper zone on layer 1, net GNDENC
- added copper zone on layer 16, net GNDENC
- added copper zone on layer 1, net GNDFAN
- added copper zone on layer 16, net GNDFAN
- added copper zone on layer 1, net GNDFAN2
- added copper zone on layer 16, net GNDFAN2
Other:
- board size 100 x 100 mm -> 84.2 x 90.1 mm
- board text added: "+"
- board text added: "-"
- board text added: "FAN"
- board text added: "HOTEND"
- board text added: "LED"
- board text added: "OPENHARDWARE.CO.ZA"
- board text added: "THERM"
- board text added: "X-CARRIAGE"
- board text added: "X-END"
- board text added: "Y-CARRIAGE"
- board text added: "Y-END"
