File: OpenHardware.co.za Controller V3.6/TestBench_rev3.6.sch (EAGLE design)
At the start: 100 parts, among them IC1 MCP2200SOIC20, IC2 ATMEGA644-20PU, IC3 7805TV, IC4 LD117ADT-TR, IC7 4050D, Q1 12Mhz, Q7 20Mhz, SW1 SPST_TACT-EVQQ2, U1 USD-SOCKETUSD, X1 USBPTH

Commit message: HY28 and Ramps1.5
Parts:
- removed BED, VMOT: (no value), con-wago-500:W237-102
- removed D6: (no value), SparkFun-DiscreteSemi:DIODESMA-ALT
- removed E1: E1, SparkFun-Connectors:M023.5MM
- removed E2: E2, SparkFun-Connectors:M023.5MM
- removed E2POL: POLOLU_A4983CARRIER, RepRapjr:POLOLU_A4983CARRIER
- removed FAN1: FAN, SparkFun-Connectors:M023.5MM
- removed JP1: (no value), jumper:JP2E
- removed JP2: (no value), SparkFun-Connectors:M04SCREW
- removed JP4: (no value), SparkFun-Connectors:M023.5MM
- removed JP6: M05X2SHD_LOCK, SparkFun-Connectors:M05X2SHD_LOCK
- removed PWRLED1, SCKLED1: (no value), LilyPad-Wearables:LED1206
- removed Q1: 12Mhz, adafruit:CRYSTALHC49UP
- removed Q3, Q4, Q5, Q6: (no value), transistor-power:PMOSFET_NTO220BV
- removed R12: 4k7, resistor:R-EU_M1206
- removed R13, R18, R21: 10R, resistor:R-EU_M1206
- removed R14: (no value), adafruit:R-US_M1206
- removed R17: (no value), SparkFun-Passives:RESISTOR1206
- removed R3: 1k, resistor:R-EU_M1206
- removed TXLED, TXLED1, VCCOK: (no value), led:LEDSMT1206
- removed X1: USBPTH, SparkFun-Connectors:USBPTH
- added 12MHZ1: (no value), crystal:CRYSTALHC49UP
- added JP10: (no value), pinhead:PINHD-2X3/90
- added LED1, LED2: (no value), adafruit:LEDSMT1206
- added U$2: CH340G, usb-serial:CH340G
- added U$3, U$4: IRLR8743, IRLR8743:IRLR8743
- added U$5: XY825A-8P, Communica.co.za:XY825A-8P
- added X2: (no value), con-berg:PN61729
- C1, C2: value 22 -> 10u; device SparkFun-Passives:CAP1206 -> rcl:CPOL-EUSANYO_SMD_B6
- C16, C17: value (none) -> 22
- C21: value 10u -> 0.1u; device rcl:CPOL-EUSANYO_SMD_B6 -> SparkFun-Passives:CAP1206
- C3, C4: value 0.1u -> 10u; device SparkFun-Passives:CAP1206 -> rcl:CPOL-EUSANYO_SMD_B6
- IC1: value MCP2200SOIC20 -> 4050D; device microchip-update-2:MCP2200SOIC20 -> 40xx:4050D
- JP18, JP19, JP20, JP5, JP7: value (none) -> M023.5MM
- R1: value 10k -> 10R
- R2: value 1k -> 10R
- U$1: value LABEL_JUMPER_1X3 -> IRLR8743; device dp_devices:LABEL_JUMPER_1X3 -> IRLR8743:IRLR8743; LEFT USB -> (none); RIGHT PSU -> (none)
Connections:
- removed net 5VREG: C30.+, IC3.VO, JP1.1
- removed net BEDOUT1: BED-1.KL, D6.A, Q3.D
- removed net BEDOUT2: D3.A, E1.2, Q5.D
- removed net DO: U1.DO
- removed net E1OUT1: D2.A, E2.2, Q4.D
- removed net E2MSFT: IC2.PCINT29/OC1A_PD5, R18.1
- removed net E2STEP: E2POL.STEP, IC2.PCINT20/TDO_PC4
- removed net EXT2ADC: C21.+, IC2.PCINT7/ADC7_PA7, JP4.2, R12.2
- removed net FANOUT1: D1.A, FAN1.2, Q6.D
- removed net N$10: R3.1, TXLED1.C
- removed net N$13: IC1.RST, R1.1
- removed net N$42: E2POL.1B, JP2.4
- removed net N$43: E2POL.1A, JP2.3
- removed net N$44: E2POL.2A, JP2.2
- removed net N$45: E2POL.2B, JP2.1
- removed net N$49: PWRLED1.A, R14.2
- removed net N$55: Q6.G, R13.2
- removed net N$61: Q4.G, R18.2
- removed net N$67: Q3.G, R21.2
- removed net N$73: JP6.8
- removed net N$9: R2.1, TXLED.C
- removed net VUSB: C4.1, IC1.VDD, JP1.3, R1.2, TXLED.A, TXLED1.A, X1.VBUS
- new net BEDOUT: D1.A, U$3.3, U$5.3
- new net D+: U$2.D+, X2.3
- new net D-: U$2.D-, X2.2
- new net EXTOUT: D3.A, U$1.3, U$5.5
- new net FANOUT: D2.A, U$4.3, U$5.7
- new net N$38: 12MHZ1.1, C16.1, U$2.XI
- new net N$40: 12MHZ1.2, C17.1, U$2.XO
- net 5V: now also U$2.VCC, X2.1; no longer C27.2, IC4.IN
- net BEDMSFT: now also R1.1; no longer R21.1
- net E1DIR: no longer E2POL.DIR
- net ENABLE: no longer E2POL.EN
- net FANMSFT: now also R2.1; no longer R13.1
- net GND: now also C1.-, C16.2, C2.-, C21.2, C3.-, C4.-, IC1P.VSS, JP10.6, LED1.C, LED2.C, U$1.1, U$2.GND, U$3.1, U$4.1, U$5.1, X2.4; no longer C1.2, C16.1, C2.1, C21.-, C3.1, C4.2, E2POL.GND@0, E2POL.GND@1, IC1.GND, JP4.1, JP6.6, PWRLED1.C, Q3.S, Q4.S, Q5.S, Q6.S, SCKLED1.C, VCCOK.C, VMOT-1.KL, X1.GND
- net MCRTS: now also U$2.DTR; no longer IC1.RTS
- net MCRX: now also U$2.RX; no longer IC1.RX
- net MCTX: now also U$2.TX; no longer IC1.TX
- net MCURESET: now also JP10.5; no longer JP6.5
- net MISO: now also JP10.1, U1.DO; no longer JP6.1
- net MOSI: now also JP10.4; no longer JP6.4
- net N$1: now also IC1B.I; no longer C2.2, IC1.OSC1, Q1.1
- net N$2: now also IC1A.I; no longer C1.1, IC1.OSC2, Q1.2
- net N$3: now also IC1A.O; no longer IC1.TXLED, R2.2
- net N$39: now also LED2.A; no longer SCKLED1.A
- net N$4: now also IC1C.I; no longer IC1.D-, X1.D-
- net N$41: now also C21.1, U$2.V3; no longer E2POL.MS1, E2POL.MS2, E2POL.MS3, R17.2
- net N$46: now also U$1.2; no longer Q5.G
- net N$5: now also IC1C.O; no longer IC1.D+, X1.D+
- net N$6: now also IC1B.O; no longer IC1.RXLED, R3.2
- net N$64: now also LED1.A; no longer VCCOK.A
- net N$7: now also R1.2, U$3.2; no longer C3.2, IC1.VUSB
- net N$8: now also R2.2, U$4.2; no longer E2POL.RST, E2POL.SLEEP
- net SCK: now also JP10.3; no longer JP6.3
- net SCL: no longer JP6.10
- net SDA: no longer JP6.9
- net SDS: no longer JP6.7
- net VCC: now also C27.2, C30.+, IC1P.VDD, IC3.VO, IC4.IN, JP10.2; no longer C17.1, E2POL.VDD, JP1.2, JP6.2, R12.1, R14.1, R17.1
- net VMOT: now also C1.+, C2.+, C3.+, C4.+, U$5.2, U$5.4, U$5.6, U$5.8; no longer BED-2.KL, C16.2, D6.C, E1.1, E2.1, E2POL.VMOT, FAN1.1, VMOT-2.KL
Other:
- note removed: "High Power DC IN"
- note removed: "Onboard SD"
- note removed: "USB-Serial"
- moved on the sheet: C16, C17, C27, C28, C30, D1, D2, D3, IC3, IC4, IC7A, IC7B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

Commit message: V3.6 with GooglePlus Interconnect Ideas
Parts:
- removed JP10: (no value), pinhead:PINHD-2X3/90
- removed JP12, JP13, JP14, JP17: (no value), SparkFun-Connectors:M04SCREW
- removed JP18, JP19, JP20: M023.5MM, SparkFun-Connectors:M023.5MM
- removed PCB1: PCB_DP_SQUARE-10X10, dp_devices:PCB_DP_SQUARE-10X10
- removed SG1: F/CM12P, buzzer:F/CM12P
- removed XENDSTOP2, YENDSTOP2, ZENDSTOP2: 22-23-2031, con-molex:22-23-2031
- added BUZZER: F/CM12P, buzzer:F/CM12P
- added C24, C26, C29: 220u, rcl:CPOL-EU153CLV-0605
- added D4, D7: (no value), dp_devices:DIODE-DO-214AC
- added IC5: (no value), linear:LM2596S
- added JP1: (no value), SparkFun-Connectors:M04LOCK
- added JP2, JP4, JP6, JP8: M05X2SHD, SparkFun-Connectors:M05X2SHD
- added L2, L3: 33uH, SparkFun-Passives:INDUCTORPWR
- added U$12: M08X2, SparkFun-Connectors:M08X2
- added U$6: CQ-121, Mantech.co.za:CQ-121
- added U$7: AVR-ISP-6-EDGE, atmega-atxmega:AVR-ISP-6-EDGE
- C25: value 100u -> 220u; device rcl:CPOL-EUE5-8.5 -> rcl:CPOL-EU153CLV-0605
- IC3: value 7805TV -> (none); device linear:7805TV -> linear:LM2596S
- R9: value (none) -> 1K
Connections:
- removed net N$2: IC1A.I
- removed net N$22: E1POL.1B, JP17.4
- removed net N$23: E1POL.1A, JP17.3
- removed net N$24: E1POL.2A, JP17.2
- removed net N$25: E1POL.2B, JP17.1
- removed net N$26: JP14.4, ZPOL.1B
- removed net N$27: JP14.3, ZPOL.1A
- removed net N$28: JP14.2, ZPOL.2A
- removed net N$29: JP14.1, ZPOL.2B
- removed net N$3: IC1A.O
- removed net N$30: JP13.1, YPOL.2B
- removed net N$31: JP13.2, YPOL.2A
- removed net N$32: JP13.3, YPOL.1A
- removed net N$33: JP13.4, YPOL.1B
- removed net N$34: JP12.4, XPOL.1B
- removed net N$35: JP12.3, XPOL.1A
- removed net N$36: JP12.2, XPOL.2A
- removed net N$37: JP12.1, XPOL.2B
- removed net N$4: IC1C.I
- removed net N$5: IC1C.O
- removed net N$6: IC1B.O
- new net 12V: C29.+, IC3.FB, JP2.9, JP4.9, JP6.9, JP8.9, L3.2, U$12.15
- new net E1A: E1POL.1A, JP8.3
- new net E1B: E1POL.1B, JP8.4
- new net E2A: E1POL.2A, JP8.2
- new net E2B: E1POL.2B, JP8.1
- new net HEATER+: U$12.5, U$12.6, U$12.7, U$12.8
- new net HEATER-: U$12.10, U$12.11, U$12.12, U$12.9
- new net N$9: D7.C, IC5.OUT, L2.1
- new net PWRIN: U$5.2, U$6.1
- new net THERMISTOR+: U$12.1, U$12.2
- new net THERMISTOR-: U$12.3, U$12.4
- new net X1A: JP4.3, XPOL.1A
- new net X1B: JP4.4, XPOL.1B
- new net X2A: JP4.2, XPOL.2A
- new net X2B: JP4.1, XPOL.2B
- new net XEND12: IC1C.I, JP4.10
- new net Y1A: JP2.3, YPOL.1A
- new net Y1B: JP2.4, YPOL.1B
- new net Y2A: JP2.2, YPOL.2A
- new net Y2B: JP2.1, YPOL.2B
- new net YEND12: IC1B.I, JP2.10
- new net Z1A: JP6.3, ZPOL.1A
- new net Z1B: JP6.4, ZPOL.1B
- new net Z2A: JP6.2, ZPOL.2A
- new net Z2B: JP6.1, ZPOL.2B
- new net ZEND12: IC1A.I, JP6.10, JP8.10, U$12.16
- net BUZZER: now also BUZZER.1; no longer SG1.1
- net GND: now also BUZZER.2, C24.-, C26.-, C29.-, D4.A, D7.A, IC3.EN, IC3.GND@1, IC5.EN, IC5.GND, IC5.GND@1, JP1.4, JP2.5, JP2.6, JP2.8, JP4.5, JP4.6, JP4.8, JP6.5, JP6.6, JP6.8, JP8.5, JP8.6, JP8.8, U$12.14, U$7.P$4; no longer JP10.6, JP18.2, JP19.2, JP20.2, SG1.2, XENDSTOP2-2.S, YENDSTOP2-2.S, ZENDSTOP2-2.S
- net MCURESET: now also U$7.P$3; no longer JP10.5
- net MISO: now also U$7.P$1; no longer JP10.1
- net MOSI: now also U$7.P$5; no longer JP10.4
- net N$1: now also D4.C, IC3.OUT, L3.1; no longer IC1B.I
- net SCK: now also U$7.P$2; no longer JP10.3
- net SCL: now also JP1.1
- net SDA: now also JP1.2
- net VCC: now also C26.+, IC5.FB, JP1.3, JP2.7, JP4.7, JP6.7, JP8.7, L2.2, U$12.13, U$7.P$6; no longer IC3.VO, JP10.2, XENDSTOP2-1.S, YENDSTOP2-1.S, ZENDSTOP2-1.S
- net VMOT: now also C24.+, IC3.IN, IC5.IN, U$6.2; no longer IC3.VI, U$5.2
- net XEND: now also IC1C.O; no longer JP20.1, XENDSTOP2-3.S
- net YEND: now also IC1B.O; no longer JP19.1, YENDSTOP2-3.S
- net ZEND: now also IC1A.O; no longer JP18.1, ZENDSTOP2-3.S
Other:
- note added: "Bed"
- note added: "CC-BY-SA 2013-2023"
- note added: "Connectors"
- note added: "E-Axis"
- note added: "Endstop Buffer"
- note added: "GooglePlus Interconnect"
- note added: "Hotend"
- note added: "Hotend Connector and Z Probe"
- note added: "Optional 12v Rail if ran from 24v"
- note added: "PSU Connector / Fuse / 5v SMPS"
- note added: "USB"
- note added: "X-Axis"
- note added: "Y-Axis"
- note added: "Z-Axis"
- note added: "and Z probe"
- note added: "uSD Socket"
- note removed: "ATX PSU Connector"
- note removed: "CC-NC 2013-2023"
- note removed: "Endstop Inputs"
- note removed: "FrontPrint"
- note removed: "High current PWR/BED"
- note removed: "I2C LCD Header"
- note removed: "ICSP Connector"
- moved on the sheet: 12MHZ1, C1, C10, C11, C12, C13, C14, C15, C16, C17, C18, C2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
