File: RAMPS1.5/RAMPS_1-3i.brd (EAGLE design)
At the start: 67 parts, among them U1 ARDUINO_MEGA_SHIELD

Commit message: Halfway through RAMPS 1.5 wishlist
Halfway through RAMPS 1.5 wishlist
Parts:
- removed C4: 100nF, capacitor-wima:C2.5-3
- removed E0-MOT, E1-MOT, X-MOT, Y-MOT, Z-MOT, Z-MOT1: (no value), RepRapjr:1X04
- removed F1: MFR500, RepRapjr:MFR500
- removed HI-AMP-OUT: DEGSON_4, Simplex-Connectors:DEGSON_4
- removed R10, R3, R5, R6, R8: 100k, adafruit:0207/7
- removed U$4, U$5, U$6, U$7, U$8: A4988BREAKOUT, RepRapjr:A4988BREAKOUT
- removed X1: (no value), con-wago-500:W237-102
- added 12V-OUT, EXT1, EXT2, FAN, HPB, PWRIN: (no value), con-wago-500:W237-102
- added C10: 470U, SparkFun-Capacitors:PANASONIC_D
- added C2, C3, C43, C7, C9: 100U, SparkFun-Capacitors:PANASONIC_D
- added C33, C34, C35, C36, C37, C38, C39, C40, C41, C42, R24, R25, R26, R27, R28: (no value), SparkFun-Passives:1206
- added DEADFUSE: (no value), led:CHIPLED_1206
- added E1POL1, E2POL1, XPOL1, YPOL1, ZPOL1: POLOLU_A4983CARRIER, RepRapjr:A4988BREAKOUT
- added F2: FUSEGSH15, fuse:GSH15
- added JP13, JP14: M023.5MM, SparkFun-Connectors:SCREWTERMINAL-3.5MM-2
- added JP15, JP16, JP17: M02PTH, SparkFun-Connectors:1X02
- added JP21, JP22, JP23, JP24, JP25: (no value), SparkFun-Connectors:SCREWTERMINAL-3.5MM-4
- added JP26: (no value), SparkFun-Connectors:1X04
- added JP27: M05X2SHD_LOCK, SparkFun-Connectors:2X5-SHROUDED_LOCK
- added JP28: (no value), SparkFun-Connectors:2X3-SHROUDED
- added R2: 1K, adafruit:M1206
- added SW1: SPST_TACT-EVQQ2, adafruit:EVQ-Q2
- C1, C5, C8: device adafruit:E2,5-5 -> adafruit:PANASONIC_C
- C6: value 470uF -> 100n; device adafruit:E3,5-8 -> SparkFun-Passives:1206
- D1, D2: value 1N4004 -> (none); device diode:DO41-10 -> adafruit:SMADIODE
- JP2, JP3, JP4, JP5, JP6: device pinhead:2X03 -> SparkFun-Connectors:1X04
- JP7: value (none) -> M023.5MM; device SparkFun:1X06 -> SparkFun-Connectors:SCREWTERMINAL-3.5MM-2
- R1, R11, R7: device adafruit:0207/7 -> adafruit:M1206
- U$1: value FSMRACD -> IRLR8743; device RepRapjr:FSMRACD -> IRLR8743:TO263
- moved D1 233.4 mm to (-175.1, 97.9)
- moved C6 227.8 mm to (-180.3, 129.5), turned to 180 degrees
- moved D2 208.1 mm to (-168.9, 96.5), turned to 90 degrees
- moved U$1 173.7 mm to (-119.4, 114.3)
- moved I2C 173.6 mm to (-39.8, -6.99), turned to 180 degrees
- moved JP6 168.1 mm to (-47.0, 137.2), turned to 180 degrees
- moved HI-AMP-IN 140.7 mm to (-181.6, 120.7), turned to 270 degrees
- moved U$11 140.6 mm to (-144.8, 114.3)
- moved JP3 137.7 mm to (-47.0, 133.3), turned to 180 degrees
- moved JP2 136.8 mm to (-63.5, 133.3), turned to 180 degrees
- moved JP5 131.0 mm to (-14.0, 133.3), turned to 180 degrees
- moved JP4 129.0 mm to (-30.5, 133.3), turned to 180 degrees
- moved U$12 126.4 mm to (-157.5, 114.3)
- moved LED1 119.4 mm to (-110.5, 64.6)
- moved U$2 118.7 mm to (-132.1, 114.3)
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Connections:
- removed net N$10: E0-MOT.3, U$4.1A
- removed net N$11: E0-MOT.4, U$4.1B
- removed net N$12: E1-MOT.1, U$5.2B
- removed net N$13: E1-MOT.2, U$5.2A
- removed net N$14: JP4.1, R5.1, U$6.MS1
- removed net N$15: JP4.3, U$6.MS2
- removed net N$16: E1-MOT.3, U$5.1A
- removed net N$17: JP5.3, U$7.MS2
- removed net N$18: E1-MOT.4, U$5.1B
- removed net N$19: JP4.5, U$6.MS3
- removed net N$20: U$6.RST, U$6.SLP
- removed net N$21: U$6.2B, X-MOT.1
- removed net N$22: U$6.2A, X-MOT.2
- removed net N$23: U$7.RST, U$7.SLP
- removed net N$24: U$5.RST, U$5.SLP
- removed net N$25: JP3.1, R3.1, U$5.MS1
- removed net N$26: U$6.1A, X-MOT.3
- removed net N$27: U$6.1B, X-MOT.4
- removed net N$28: U$7.2B, Y-MOT.1
- removed net N$29: U$7.2A, Y-MOT.2
- removed net N$30: U$7.1A, Y-MOT.3
- removed net N$31: JP5.5, U$7.MS3
- removed net N$33: JP5.1, R8.1, U$7.MS1
- removed net N$34: JP3.5, U$5.MS3
- removed net N$35: JP3.3, U$5.MS2
- removed net N$36: U$7.1B, Y-MOT.4
- removed net N$37: JP6.3, U$8.MS2
- removed net N$38: U$8.RST, U$8.SLP
- removed net N$39: JP6.5, U$8.MS3
- removed net N$40: JP6.1, R10.1, U$8.MS1
- removed net N$41: U$8.2B, Z-MOT.1, Z-MOT1.1
- removed net N$42: U$8.2A, Z-MOT.2, Z-MOT1.2
- removed net N$43: U$8.1A, Z-MOT.3, Z-MOT1.3
- removed net N$44: U$8.1B, Z-MOT.4, Z-MOT1.4
- removed net N$6: JP2.5, U$4.MS3
- removed net N$8: U$4.RST, U$4.SLP
- removed net N$9: JP2.3, U$4.MS2
- new net +24V: EXT1.2, EXT2.2, HPB.2
- new net ENCA: JP28.2
- new net ENCB: JP28.3
- new net ENCC: JP28.4
- new net FANPIN: U$1.1
- new net MCURESET: JP27.5
- new net N$52: E1POL1.RST, E1POL1.SLP
- new net N$53: ZPOL1.RST, ZPOL1.SLP
- new net N$56: YPOL1.RST, YPOL1.SLP
- new net N$57: XPOL1.RST, XPOL1.SLP
- new net N$58: R26.2, XPOL1.MS1, XPOL1.MS2, XPOL1.MS3
- new net N$59: R24.2, YPOL1.MS1, YPOL1.MS2, YPOL1.MS3
- new net N$60: E1POL1.MS1, E1POL1.MS2, E1POL1.MS3, R27.2
- new net N$62: R25.2, ZPOL1.MS1, ZPOL1.MS2, ZPOL1.MS3
- new net N$63: E1POL1.1B, JP24.4, JP4.4
- new net N$65: E1POL1.1A, JP24.3, JP4.3
- new net N$66: JP27.8
- new net N$68: E1POL1.2A, JP24.2, JP4.2
- new net N$69: E1POL1.2B, JP24.1, JP4.1
- new net N$70: JP23.4, JP3.4, JP6.4, ZPOL1.1B
- new net N$71: JP23.3, JP3.3, JP6.3, ZPOL1.1A
- new net N$72: JP23.2, JP3.2, JP6.2, ZPOL1.2A
- new net N$74: JP23.1, JP3.1, JP6.1, ZPOL1.2B
- new net N$75: JP2.1, JP22.1, YPOL1.2B
- new net N$76: JP2.2, JP22.2, YPOL1.2A
- new net N$77: JP2.3, JP22.3, YPOL1.1A
- new net N$78: JP2.4, JP22.4, YPOL1.1B
- new net N$79: JP21.4, JP26.4, XPOL1.1B
- new net N$80: JP21.3, JP26.3, XPOL1.1A
- new net N$81: JP21.2, JP26.2, XPOL1.2A
- new net N$82: JP21.1, JP26.1, XPOL1.2B
- new net N$83: E2POL1.RST, E2POL1.SLP
- new net N$84: E2POL1.MS1, E2POL1.MS2, E2POL1.MS3, R28.2
- new net N$85: E2POL1.1B, JP25.4, JP5.4
- new net N$86: E2POL1.1A, JP25.3, JP5.3
- new net N$87: E2POL1.2A, JP25.2, JP5.2
- new net N$88: E2POL1.2B, JP25.1, JP5.1
- new net SDS: JP27.7
- new net VMOT: C2.+, C3.+, C34.2, C36.2, C37.2, C40.2, C41.2, C43.+, C7.+, C9.+, E1POL1.VMOT, E2POL1.VMOT, XPOL1.VMOT, YPOL1.VMOT, ZPOL1.VMOT
- net +12V: now also 12V-OUT.1, C10.+, C6.2, FAN.2; no longer C4.1, C6.+, D2.C, F1.1, HI-AMP-OUT.1, HI-AMP-OUT.3, U$4.VMOT, U$5.VMOT, U$6.VMOT, U$7.VMOT, U$8.VMOT, X1.2
- net E0-DIR: now also E1POL1.DIR; no longer U$4.DIR
- net E0-EN: now also E1POL1.EN; no longer U$4.EN
- net E0-STEP: now also E1POL1.STEP; no longer U$4.STEP
- net E1-DIR: now also E2POL1.DIR; no longer U$5.DIR
- net E1-EN: now also E2POL1.EN; no longer U$5.EN
- net E1-STEP: now also E2POL1.STEP; no longer U$5.STEP
- net GND: now also 12V-OUT.2, C10.-, C2.-, C3.-, C33.2, C34.1, C35.2, C36.1, C37.1, C38.2, C39.2, C40.1, C41.1, C42.2, C43.-, C6.1, C7.-, C9.-, E1POL1.GND, E1POL1.GND@0, E2POL1.GND, E2POL1.GND@0, JP13.1, JP14.1, JP15.1, JP16.1, JP17.1, JP27.6, JP28.1, JP28.5, PWRIN.2, SW1.A, SW1.A', U$1.2, XPOL1.GND, XPOL1.GND@0, YPOL1.GND, YPOL1.GND@0, ZPOL1.GND, ZPOL1.GND@0; no longer C4.2, C6.-, JP7.3, JP7.5, R10.2, R3.2, R5.2, R6.1, R8.2, U$1.GND1, U$1.GND2, U$1.P$1, U$4.GND, U$4.GND@0, U$5.GND, U$5.GND@0, U$6.GND, U$6.GND@0, U$7.GND, U$7.GND@0, U$8.GND, U$8.GND@0
- net MISO: now also JP27.1
- net MOSI: now also JP27.4
- net N$1: now also EXT2.1; no longer X1.1
- net N$2: now also HPB.1; no longer HI-AMP-OUT.4
- net N$3: now also DEADFUSE.A, R2.1; no longer E0-MOT.1, U$4.2B
- net N$32: now also F2.1, PWRIN.1, R2.2; no longer F1.2
- net N$4: now also D2.C, DEADFUSE.C, F2.2; no longer E0-MOT.2, U$4.2A
- net N$47: now also EXT1.1; no longer HI-AMP-OUT.2
- net N$5: now also FAN.1, U$1.3; no longer JP2.1, R6.2, U$4.MS1
- net RESET: now also SW1.B, SW1.B'; no longer U$1.P$2
- net SCK: now also JP27.3
- net SCL: now also JP27.10
- net SDA: now also JP27.9
- net THERM0: now also JP15.2
- net THERM1: now also JP13.2, JP16.2; no longer JP7.4
- net THERM2: now also JP14.2, JP17.2; no longer JP7.6
- net VCC: now also C33.1, C35.1, C38.1, C39.1, C42.1, E1POL1.VDD, E2POL1.VDD, JP27.2, JP28.6, R24.1, R25.1, R26.1, R27.1, R28.1, XPOL1.VDD, YPOL1.VDD, ZPOL1.VDD; no longer JP2.2, JP2.4, JP2.6, JP3.2, JP3.4, JP3.6, JP4.2, JP4.4, JP4.6, JP5.2, JP5.4, JP5.6, JP6.2, JP6.4, JP6.6, U$4.VDD, U$5.VDD, U$6.VDD, U$7.VDD, U$8.VDD
- net X-DIR: now also XPOL1.DIR; no longer U$6.DIR
- net X-EN: now also XPOL1.EN; no longer U$6.EN
- net X-STEP: now also XPOL1.STEP; no longer U$6.STEP
- net Y-DIR: now also YPOL1.DIR; no longer U$7.DIR
- net Y-EN: now also YPOL1.EN; no longer U$7.EN
- net Y-STEP: now also YPOL1.STEP; no longer U$7.STEP
- net Z-DIR: now also ZPOL1.DIR; no longer U$8.DIR
- net Z-EN: now also ZPOL1.EN; no longer U$8.EN
- net Z-STEP: now also ZPOL1.STEP; no longer U$8.STEP
Routing:
- net VCC: track 340.2 -> 0.00 mm
- net GND: track 189.7 -> 0.00 mm
- net +12V: track 125.9 -> 0.00 mm
- net D1: track 84.1 -> 0.00 mm
- net D2: track 83.1 -> 0.00 mm
- net X-EN: track 78.5 -> 0.00 mm
- net E0-EN: track 68.1 -> 0.00 mm
- net D6: track 65.5 -> 0.00 mm
- net D4: track 62.8 -> 0.00 mm
- net D7: track 62.7 -> 0.00 mm
- net D5: track 62.5 -> 0.00 mm
- net E0-STEP: track 54.3 -> 0.00 mm
- net THERM0: track 53.6 -> 0.00 mm
- net D12: track 52.7 -> 0.00 mm
- net E0-DIR: track 50.9 -> 0.00 mm
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- added copper zone on layer 1, net 5V
Other:
- board text added: "Done: Added FAN Mosfet Added 12v RAIL (TODO: Switchmode from 24v) Added fuse with blown indicator LED Added 3.5mm screw terminals in parallel to 0.1" headers for motors, endstops, thermistors Added D size SMD caps (63v) to VMOTOR for each driver Added D size SMD cap for 470u on 12v rail Changed Thermistor to C-Type SMD 10u Caps and 1206 4k7 Resistors Kept original servo and expansion headers in e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"
- board text added: "E0"
- board text added: "E1"
- board text added: "ENDSTOPS"
- board text added: "Pwr, Mosfets, Fuse, Fuse-dead-LED"
- board text added: "Stepper Drivers"
- board text added: "Thermistors"
- board text added: "To-Do Design 24v rail Add switchmode converter to feed 12v rail Find proper terminals for high current connections - parallel footprint with 5mm screw terminals Add back SJ's for Microstepping Add flyback diodes on MOSFETs for safety Add Z Probe circuitry Request: Add small FDC8886's to switch 12v for other fans, LEDs, etc If space left over investigate PT100s Fix footprint for fuse to correct AT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"
- board text added: "Y"
- board text added: "Z"
- board text added: "therm0"
- board text added: "therm1"
- board text added: "therm2"
- board text added: "x"
- board text added: "xmax"
- board text added: "xmin"
- board text added: "ymax"
- board text added: "ymin"
- board text added: "zmax"
- board text added: "zmin"

Commit message: HY28 and Ramps1.5
Parts:
- removed HI-AMP-IN: DEGSON_2, Simplex-Connectors:DEGSON_2
- removed JP27: M05X2SHD_LOCK, SparkFun-Connectors:2X5-SHROUDED_LOCK
- removed JP28: (no value), SparkFun-Connectors:2X3-SHROUDED
- added C11: 100n, SparkFun-Passives:1206
- added C4: 470U, SparkFun-Capacitors:PANASONIC_D
- added D3, D4, D5, D6: (no value), adafruit:SMADIODE
- added JP18: (no value), SparkFun-Connectors:SCREWTERMINAL-3.5MM-3_LOCK.007S
- added R3: 15K, adafruit:M1206
- added R4: 10K, adafruit:M1206
- added SJ1, SJ10, SJ11, SJ12, SJ13, SJ14, SJ15, SJ2, SJ3, SJ4, SJ5, SJ6, SJ7, SJ8, SJ9: (no value), jumper:SJ
- added U$4: XY825A-8P, Communica.co.za:XY825A-8P
- added Z+1: (no value), ultimachine:3PIN-HEADER
- R12: device adafruit:0207/7 -> adafruit:M1206
- moved DEADFUSE 58.8 mm to (-204.5, 102.9), turned to 180 degrees
- moved R2 52.7 mm to (-204.5, 110.5), turned to 90 degrees
- moved F2 47.3 mm to (-196.8, 105.4), turned to 270 degrees
- moved I2C 31.1 mm to (-13.5, 9.53), turned to 0 degrees
- moved EXT2 24.7 mm to (-120.7, 134.6)
- moved C6 23.9 mm to (-190.5, 108.0), turned to 90 degrees
- moved EXT1 22.2 mm to (-135.9, 134.6)
- moved U$11 21.8 mm to (-127.0, 101.6)
- moved U$1 19.8 mm to (-104.1, 101.6)
- moved FAN 19.8 mm to (-104.1, 116.8)
- moved HPB 19.7 mm to (-151.1, 134.6)
- moved PWRIN 18.9 mm to (-165.1, 133.3), turned to 180 degrees
- moved D2 17.8 mm to (-186.7, 95.2), turned to 270 degrees
- moved 12V-OUT 17.1 mm to (-180.3, 116.8)
- moved U$2 14.8 mm to (-139.7, 101.6)
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Connections:
- removed net ENCA: JP28.2
- removed net ENCB: JP28.3
- removed net ENCC: JP28.4
- removed net MCURESET: JP27.5
- removed net N$1: EXT2.1, U$11.3
- removed net N$2: HPB.1, U$2.3
- removed net N$32: F2.1, HI-AMP-IN.2, PWRIN.1, R2.2
- removed net N$47: EXT1.1, U$12.3
- removed net N$5: FAN.1, U$1.3
- removed net N$66: JP27.8
- removed net SDS: JP27.7
- new net 12V: JP18.1, Z+1.1
- new net BEDOUT: D3.A, HPB.1, U$2.3, U$4.3
- new net E1OUT: D4.A, EXT1.1, U$12.3, U$4.5
- new net E2OUT: D5.A, EXT2.1, U$11.3, U$4.7
- new net FANOUT: D6.A, FAN.1, U$1.3
- new net N$10: SJ8.2, ZPOL1.MS2
- new net N$11: SJ9.2, ZPOL1.MS3
- new net N$12: SJ6.2, YPOL1.MS3
- new net N$13: SJ3.2, XPOL1.MS3
- new net N$14: E2POL1.MS2, SJ14.2
- new net N$15: E2POL1.MS3, SJ13.2
- new net N$16: E2POL1.MS1, SJ15.2
- new net N$17: E1POL1.MS3, SJ12.2
- new net N$18: E1POL1.MS1, SJ10.2
- new net N$19: E1POL1.MS2, SJ11.2
- new net N$6: SJ1.2, XPOL1.MS1
- new net N$7: SJ4.2, YPOL1.MS1
- new net N$8: SJ5.2, YPOL1.MS2
- new net N$9: SJ7.2, ZPOL1.MS1
- new net PWRIN: F2.1, PWRIN.1, R2.2, U$4.2
- new net SENSOROUT: JP18.2, R3.1, Z+1.2
- net +12V: now also D6.C
- net +24V: now also C11.2, C4.+, D2.C, D3.C, D4.C, D5.C, DEADFUSE.C, F2.2, U$4.6, U$4.8
- net GND: now also C11.1, C4.-, JP18.3, R4.1, U$4.1, Z+1.3; no longer HI-AMP-IN.1, JP27.6, JP28.1, JP28.5
- net MISO: no longer JP27.1
- net MOSI: no longer JP27.4
- net N$4: now also SJ2.2, XPOL1.MS2; no longer D2.C, DEADFUSE.C, F2.2
- net N$58: now also SJ1.1, SJ2.1, SJ3.1; no longer XPOL1.MS1, XPOL1.MS2, XPOL1.MS3
- net N$59: now also SJ4.1, SJ5.1, SJ6.1; no longer YPOL1.MS1, YPOL1.MS2, YPOL1.MS3
- net N$60: now also SJ10.1, SJ11.1, SJ12.1; no longer E1POL1.MS1, E1POL1.MS2, E1POL1.MS3
- net N$62: now also SJ7.1, SJ8.1, SJ9.1; no longer ZPOL1.MS1, ZPOL1.MS2, ZPOL1.MS3
- net N$84: now also SJ13.1, SJ14.1, SJ15.1; no longer E2POL1.MS1, E2POL1.MS2, E2POL1.MS3
- net SCK: no longer JP27.3
- net SCL: no longer JP27.10
- net SDA: no longer JP27.9
- net VCC: no longer JP27.2, JP28.6
- net Z-MIN: now also R3.2, R4.2
Other:
- board text added: "To-Do Add switchmode converter to feed 12v rail Request: Add small FDC8886's to switch 12v for other fans, LEDs, etc If space left over investigate PT100s Fix footprint for fuse to correct ATQ Automotive fuse"
- board text added: "Z-Probe"
- board text removed: "To-Do Design 24v rail Add switchmode converter to feed 12v rail Find proper terminals for high current connections - parallel footprint with 5mm screw terminals Add back SJ's for Microstepping Add flyback diodes on MOSFETs for safety Add Z Probe circuitry Request: Add small FDC8886's to switch 12v for other fans, LEDs, etc If space left over investigate PT100s Fix footprint for fuse to correct AT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"

Commit message: V3.6 with GooglePlus Interconnect Ideas
Parts:
- removed F2: FUSEGSH15, fuse:GSH15
- added C12, C13: 220u, rcl:153CLV-0605
- added D7: (no value), dp_devices:DO-214AC
- added IC1: (no value), linear:TO263-5
- added L1: (no value), SparkFun-Passives:CDRH125
- added U$5: CQ-121, Mantech.co.za:CQ121
- moved JP18 40.6 mm to (-269.2, 118.1)
- moved R3 40.6 mm to (-265.4, 111.8)
- moved R4 40.6 mm to (-261.6, 111.8)
- moved Z+1 40.6 mm to (-266.7, 121.9)
- moved DEADFUSE 21.3 mm to (-198.1, 123.2)
- moved R2 20.1 mm to (-198.1, 129.5)
- moved FAN 17.8 mm to (-104.1, 134.6)
- moved 12V-OUT 16.7 mm to (-182.9, 133.3), turned to 180 degrees
- moved PWRIN 2.54 mm to (-167.6, 133.3)
- moved D1 1.27 mm to (-185.5, 106.9)
- moved D2 1.27 mm to (-185.4, 95.2)
- moved I2C 1.27 mm to (-14.8, 9.53)
- moved C11 1.27 mm to (-190.5, 95.2)
- moved C6 1.27 mm to (-190.5, 106.7)
- moved D6 1.27 mm to (-104.1, 113.0), turned to 180 degrees
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Connections:
- new net N$1: D7.1, IC1.2, L1.1
- net +12V: now also C13.+, IC1.4, L1.2
- net +24V: now also C12.+, IC1.1, U$5.3@2, U$5.4@2; no longer F2.2
- net GND: now also C12.-, C13.-, D7.2, IC1.3, IC1.5, IC1.6
- net PWRIN: now also U$5.1@1, U$5.2@1; no longer F2.1
Other:
- board text added: "24-12v SMPS"
- board text added: "To-Do Add switchmode converter to feed 12v rail Request: Add small FDC8886's to switch 12v for other fans, LEDs, etc If space left over investigate PT100s"
- board text removed: "To-Do Add switchmode converter to feed 12v rail Request: Add small FDC8886's to switch 12v for other fans, LEDs, etc If space left over investigate PT100s Fix footprint for fuse to correct ATQ Automotive fuse"
