File: RAMPS1.5/RAMPS_1-3i.sch (EAGLE design)
At the start: 67 parts, among them U1 ARDUINO_MEGA_SHIELD

Commit message: Halfway through RAMPS 1.5 wishlist
Halfway through RAMPS 1.5 wishlist
Parts:
- removed C4: 100nF, capacitor-wima:C2,5-3
- removed E0-MOT, E1-MOT, X-MOT, Y-MOT, Z-MOT, Z-MOT1: (no value), RepRapjr:PINHD-1X4
- removed F1: MFR500, RepRapjr:PTCFUSE
- removed HI-AMP-OUT: DEGSON_4, Simplex-Connectors:DEGSON_4
- removed R10, R3, R5, R6, R8: 100k, adafruit:R-US_0207/7
- removed U$4, U$5, U$6, U$7, U$8: A4988BREAKOUT, RepRapjr:A4988BREAKOUT
- removed X1: (no value), con-wago-500:W237-102
- added 12V-OUT, EXT1, EXT2, FAN, HPB, PWRIN: (no value), con-wago-500:W237-102
- added C10: 470U, SparkFun-Capacitors:CAP_POLD
- added C2, C3, C43, C7, C9: 100U, SparkFun-Capacitors:CAP_POLD
- added C33, C34, C35, C36, C37, C38, C39, C40, C41, C42: (no value), SparkFun-Passives:CAP1206
- added DEADFUSE: (no value), led:LEDCHIPLED_1206
- added E1POL1, E2POL1, XPOL1, YPOL1, ZPOL1: POLOLU_A4983CARRIER, RepRapjr:POLOLU_A4983CARRIER
- added F2: FUSEGSH15, fuse:FUSEGSH15
- added JP13, JP14: M023.5MM, SparkFun-Connectors:M023.5MM
- added JP15, JP16, JP17: M02PTH, SparkFun-Connectors:M02PTH
- added JP21, JP22, JP23, JP24, JP25: (no value), SparkFun-Connectors:M04SCREW
- added JP26: (no value), SparkFun-Connectors:M04PTH
- added JP27: M05X2SHD_LOCK, SparkFun-Connectors:M05X2SHD_LOCK
- added JP28: (no value), SparkFun-Connectors:M03X2SHROUD
- added R2: 1K, adafruit:R-US_M1206
- added R24, R25, R26, R27, R28: (no value), SparkFun-Passives:RESISTOR1206
- added SW1: SPST_TACT-EVQQ2, adafruit:SPST_TACT-EVQQ2
- C1, C5, C8: device adafruit:CPOL-USE2.5-5 -> adafruit:CPOL-USC
- C6: value 470uF -> 100n; device adafruit:CPOL-USE3.5-8 -> SparkFun-Passives:CAP1206
- D1, D2: value 1N4004 -> (none); device diode:1N4004 -> adafruit:DIODESMA
- JP2, JP3, JP4, JP5, JP6: device pinhead:PINHD-2X3 -> SparkFun-Connectors:M04PTH
- JP7: value (none) -> M023.5MM; device SparkFun:M06SIP -> SparkFun-Connectors:M023.5MM
- R1, R11, R7: device adafruit:R-US_0207/7 -> adafruit:R-US_M1206
- U$1: value FSMRACD -> IRLR8743; device RepRapjr:FSMRACD -> IRLR8743:IRLR8743
Connections:
- removed net N$10: E0-MOT.3, U$4.1A
- removed net N$11: E0-MOT.4, U$4.1B
- removed net N$12: E1-MOT.1, U$5.2B
- removed net N$13: E1-MOT.2, U$5.2A
- removed net N$14: JP4.1, R5.1, U$6.MS1
- removed net N$15: JP4.3, U$6.MS2
- removed net N$16: E1-MOT.3, U$5.1A
- removed net N$17: JP5.3, U$7.MS2
- removed net N$18: E1-MOT.4, U$5.1B
- removed net N$19: JP4.5, U$6.MS3
- removed net N$20: U$6.RST, U$6.SLEEP
- removed net N$21: U$6.2B, X-MOT.1
- removed net N$22: U$6.2A, X-MOT.2
- removed net N$23: U$7.RST, U$7.SLEEP
- removed net N$24: U$5.RST, U$5.SLEEP
- removed net N$25: JP3.1, R3.1, U$5.MS1
- removed net N$26: U$6.1A, X-MOT.3
- removed net N$27: U$6.1B, X-MOT.4
- removed net N$28: U$7.2B, Y-MOT.1
- removed net N$29: U$7.2A, Y-MOT.2
- removed net N$30: U$7.1A, Y-MOT.3
- removed net N$31: JP5.5, U$7.MS3
- removed net N$33: JP5.1, R8.1, U$7.MS1
- removed net N$34: JP3.5, U$5.MS3
- removed net N$35: JP3.3, U$5.MS2
- removed net N$36: U$7.1B, Y-MOT.4
- removed net N$37: JP6.3, U$8.MS2
- removed net N$38: U$8.RST, U$8.SLEEP
- removed net N$39: JP6.5, U$8.MS3
- removed net N$40: JP6.1, R10.1, U$8.MS1
- removed net N$41: U$8.2B, Z-MOT.1, Z-MOT1.1
- removed net N$42: U$8.2A, Z-MOT.2, Z-MOT1.2
- removed net N$43: U$8.1A, Z-MOT.3, Z-MOT1.3
- removed net N$44: U$8.1B, Z-MOT.4, Z-MOT1.4
- removed net N$6: JP2.5, U$4.MS3
- removed net N$8: U$4.RST, U$4.SLEEP
- removed net N$9: JP2.3, U$4.MS2
- new net +24V: EXT1-2.KL, EXT2-2.KL, HPB-2.KL
- new net ENCA: JP28.2
- new net ENCB: JP28.3
- new net ENCC: JP28.4
- new net FANPIN: U$1.2
- new net MCURESET: JP27.5
- new net N$52: E1POL1.RST, E1POL1.SLEEP
- new net N$53: ZPOL1.RST, ZPOL1.SLEEP
- new net N$56: YPOL1.RST, YPOL1.SLEEP
- new net N$57: XPOL1.RST, XPOL1.SLEEP
- new net N$58: R26.2, XPOL1.MS1, XPOL1.MS2, XPOL1.MS3
- new net N$59: R24.2, YPOL1.MS1, YPOL1.MS2, YPOL1.MS3
- new net N$60: E1POL1.MS1, E1POL1.MS2, E1POL1.MS3, R27.2
- new net N$62: R25.2, ZPOL1.MS1, ZPOL1.MS2, ZPOL1.MS3
- new net N$63: E1POL1.1B, JP24.4, JP4.4
- new net N$65: E1POL1.1A, JP24.3, JP4.3
- new net N$66: JP27.8
- new net N$68: E1POL1.2A, JP24.2, JP4.2
- new net N$69: E1POL1.2B, JP24.1, JP4.1
- new net N$70: JP23.4, JP3.4, JP6.4, ZPOL1.1B
- new net N$71: JP23.3, JP3.3, JP6.3, ZPOL1.1A
- new net N$72: JP23.2, JP3.2, JP6.2, ZPOL1.2A
- new net N$74: JP23.1, JP3.1, JP6.1, ZPOL1.2B
- new net N$75: JP2.1, JP22.1, YPOL1.2B
- new net N$76: JP2.2, JP22.2, YPOL1.2A
- new net N$77: JP2.3, JP22.3, YPOL1.1A
- new net N$78: JP2.4, JP22.4, YPOL1.1B
- new net N$79: JP21.4, JP26.4, XPOL1.1B
- new net N$80: JP21.3, JP26.3, XPOL1.1A
- new net N$81: JP21.2, JP26.2, XPOL1.2A
- new net N$82: JP21.1, JP26.1, XPOL1.2B
- new net N$83: E2POL1.RST, E2POL1.SLEEP
- new net N$84: E2POL1.MS1, E2POL1.MS2, E2POL1.MS3, R28.2
- new net N$85: E2POL1.1B, JP25.4, JP5.4
- new net N$86: E2POL1.1A, JP25.3, JP5.3
- new net N$87: E2POL1.2A, JP25.2, JP5.2
- new net N$88: E2POL1.2B, JP25.1, JP5.1
- new net SDS: JP27.7
- new net VMOT: C2.+, C3.+, C34.2, C36.2, C37.2, C40.2, C41.2, C43.+, C7.+, C9.+, E1POL1.VMOT, E2POL1.VMOT, XPOL1.VMOT, YPOL1.VMOT, ZPOL1.VMOT
- net +12V: now also 12V-OUT-1.KL, C10.+, C6.2, FAN-2.KL; no longer C4.1, C6.+, D2.C, F1.1, HI-AMP-OUTG$1.KL, HI-AMP-OUTG$3.KL, U$4.VMOT, U$5.VMOT, U$6.VMOT, U$7.VMOT, U$8.VMOT, X1-2.KL
- net E0-DIR: now also E1POL1.DIR; no longer U$4.DIR
- net E0-EN: now also E1POL1.EN; no longer U$4.EN
- net E0-STEP: now also E1POL1.STEP; no longer U$4.STEP
- net E1-DIR: now also E2POL1.DIR; no longer U$5.DIR
- net E1-EN: now also E2POL1.EN; no longer U$5.EN
- net E1-STEP: now also E2POL1.STEP; no longer U$5.STEP
- net GND: now also 12V-OUT-2.KL, C10.-, C2.-, C3.-, C33.2, C34.1, C35.2, C36.1, C37.1, C38.2, C39.2, C40.1, C41.1, C42.2, C43.-, C6.1, C7.-, C9.-, E1POL1.GND@0, E1POL1.GND@1, E2POL1.GND@0, E2POL1.GND@1, JP13.1, JP14.1, JP15.1, JP16.1, JP17.1, JP27.6, JP28.1, JP28.5, PWRIN-2.KL, SW1.P, SW1.P1, U$1.1, XPOL1.GND@0, XPOL1.GND@1, YPOL1.GND@0, YPOL1.GND@1, ZPOL1.GND@0, ZPOL1.GND@1; no longer C4.2, C6.-, JP7.3, JP7.5, R10.2, R3.2, R5.2, R6.1, R8.2, U$1.GND1, U$1.GND2, U$1.P, U$4.GND@0, U$4.GND@1, U$5.GND@0, U$5.GND@1, U$6.GND@0, U$6.GND@1, U$7.GND@0, U$7.GND@1, U$8.GND@0, U$8.GND@1
- net MISO: now also JP27.1
- net MOSI: now also JP27.4
- net N$1: now also EXT2-1.KL; no longer X1-1.KL
- net N$2: now also HPB-1.KL; no longer HI-AMP-OUTG$4.KL
- net N$3: now also DEADFUSE.A, R2.1; no longer E0-MOT.1, U$4.2B
- net N$32: now also F2.1, PWRIN-1.KL, R2.2; no longer F1.2
- net N$4: now also D2.C, DEADFUSE.C, F2.2; no longer E0-MOT.2, U$4.2A
- net N$47: now also EXT1-1.KL; no longer HI-AMP-OUTG$2.KL
- net N$5: now also FAN-1.KL, U$1.3; no longer JP2.1, R6.2, U$4.MS1
- net RESET: now also SW1.S, SW1.S1; no longer U$1.S
- net SCK: now also JP27.3
- net SCL: now also JP27.10
- net SDA: now also JP27.9
- net THERM0: now also JP15.2
- net THERM1: now also JP13.2, JP16.2; no longer JP7.4
- net THERM2: now also JP14.2, JP17.2; no longer JP7.6
- net VCC: now also C33.1, C35.1, C38.1, C39.1, C42.1, E1POL1.VDD, E2POL1.VDD, JP27.2, JP28.6, R24.1, R25.1, R26.1, R27.1, R28.1, XPOL1.VDD, YPOL1.VDD, ZPOL1.VDD; no longer JP2.2, JP2.4, JP2.6, JP3.2, JP3.4, JP3.6, JP4.2, JP4.4, JP4.6, JP5.2, JP5.4, JP5.6, JP6.2, JP6.4, JP6.6, U$4.VDD, U$5.VDD, U$6.VDD, U$7.VDD, U$8.VDD
- net X-DIR: now also XPOL1.DIR; no longer U$6.DIR
- net X-EN: now also XPOL1.EN; no longer U$6.EN
- net X-STEP: now also XPOL1.STEP; no longer U$6.STEP
- net Y-DIR: now also YPOL1.DIR; no longer U$7.DIR
- net Y-EN: now also YPOL1.EN; no longer U$7.EN
- net Y-STEP: now also YPOL1.STEP; no longer U$7.STEP
- net Z-DIR: now also ZPOL1.DIR; no longer U$8.DIR
- net Z-EN: now also ZPOL1.EN; no longer U$8.EN
- net Z-STEP: now also ZPOL1.STEP; no longer U$8.STEP
Other:
- note added: "12v-out"
- note added: "E3D Fan for example"
- note added: "PWR For Atmega from 12v rail"
- note added: "UI CONNECTORS"
- note removed: "TODO: Replace with ATQ Stylke fuse"

Commit message: HY28 and Ramps1.5
Parts:
- removed HI-AMP-IN: DEGSON_2, Simplex-Connectors:DEGSON_2
- removed JP27: M05X2SHD_LOCK, SparkFun-Connectors:M05X2SHD_LOCK
- removed JP28: (no value), SparkFun-Connectors:M03X2SHROUD
- added C11: 100n, SparkFun-Passives:CAP1206
- added C4: 470U, SparkFun-Capacitors:CAP_POLD
- added D3, D4, D5, D6: (no value), adafruit:DIODESMA
- added JP18: (no value), SparkFun-Connectors:M03SCREW_LOCK
- added R3: 15K, adafruit:R-US_M1206
- added R4: 10K, adafruit:R-US_M1206
- added SJ1, SJ10, SJ11, SJ12, SJ13, SJ14, SJ15, SJ2, SJ3, SJ4, SJ5, SJ6, SJ7, SJ8, SJ9: (no value), jumper:SJ
- added U$4: XY825A-8P, Communica.co.za:XY825A-8P
- added Z+1: (no value), ultimachine:3PIN-HEADER
- R12: device adafruit:R-US_0207/7 -> adafruit:R-US_M1206
Connections:
- removed net ENCA: JP28.2
- removed net ENCB: JP28.3
- removed net ENCC: JP28.4
- removed net MCURESET: JP27.5
- removed net N$1: EXT2-1.KL, U$11.3
- removed net N$2: HPB-1.KL, U$2.3
- removed net N$32: F2.1, HI-AMP-ING$2.KL, PWRIN-1.KL, R2.2
- removed net N$47: EXT1-1.KL, U$12.3
- removed net N$5: FAN-1.KL, U$1.3
- removed net N$66: JP27.8
- removed net SDS: JP27.7
- new net 12V: JP18.1, Z+1.1
- new net BEDOUT: D3.A, HPB-1.KL, U$2.3, U$4.3
- new net E1OUT: D4.A, EXT1-1.KL, U$12.3, U$4.5
- new net E2OUT: D5.A, EXT2-1.KL, U$11.3, U$4.7
- new net FANOUT: D6.A, FAN-1.KL, U$1.3
- new net N$10: SJ8.2, ZPOL1.MS2
- new net N$11: SJ9.2, ZPOL1.MS3
- new net N$12: SJ6.2, YPOL1.MS3
- new net N$13: SJ3.2, XPOL1.MS3
- new net N$14: E2POL1.MS2, SJ14.2
- new net N$15: E2POL1.MS3, SJ13.2
- new net N$16: E2POL1.MS1, SJ15.2
- new net N$17: E1POL1.MS3, SJ12.2
- new net N$18: E1POL1.MS1, SJ10.2
- new net N$19: E1POL1.MS2, SJ11.2
- new net N$6: SJ1.2, XPOL1.MS1
- new net N$7: SJ4.2, YPOL1.MS1
- new net N$8: SJ5.2, YPOL1.MS2
- new net N$9: SJ7.2, ZPOL1.MS1
- new net PWRIN: F2.1, PWRIN-1.KL, R2.2, U$4.2
- new net SENSOROUT: JP18.2, R3.1, Z+1.2
- net +12V: now also D6.C
- net +24V: now also C11.2, C4.+, D2.C, D3.C, D4.C, D5.C, DEADFUSE.C, F2.2, U$4.6, U$4.8
- net GND: now also C11.1, C4.-, JP18.3, R4.1, U$4.1, Z+1.3; no longer HI-AMP-ING$1.KL, JP27.6, JP28.1, JP28.5
- net MISO: no longer JP27.1
- net MOSI: no longer JP27.4
- net N$4: now also SJ2.2, XPOL1.MS2; no longer D2.C, DEADFUSE.C, F2.2
- net N$58: now also SJ1.1, SJ2.1, SJ3.1; no longer XPOL1.MS1, XPOL1.MS2, XPOL1.MS3
- net N$59: now also SJ4.1, SJ5.1, SJ6.1; no longer YPOL1.MS1, YPOL1.MS2, YPOL1.MS3
- net N$60: now also SJ10.1, SJ11.1, SJ12.1; no longer E1POL1.MS1, E1POL1.MS2, E1POL1.MS3
- net N$62: now also SJ7.1, SJ8.1, SJ9.1; no longer ZPOL1.MS1, ZPOL1.MS2, ZPOL1.MS3
- net N$84: now also SJ13.1, SJ14.1, SJ15.1; no longer E2POL1.MS1, E2POL1.MS2, E2POL1.MS3
- net SCK: no longer JP27.3
- net SCL: no longer JP27.10
- net SDA: no longer JP27.9
- net VCC: no longer JP27.2, JP28.6
- net Z-MIN: now also R3.2, R4.2
Other:
- note added: "GND"
- note added: "OUT"
- note added: "VIN"
- note added: "Z-Probe"
- note removed: "UI CONNECTORS"
- moved on the sheet: 12V-OUT-1, 12V-OUT-2, 5V, C10, C6, D1, D2, DEADFUSE, EXT1-1, EXT1-2, EXT2-1, EXT2-2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

Commit message: V3.6 with GooglePlus Interconnect Ideas
Parts:
- removed F2: FUSEGSH15, fuse:FUSEGSH15
- added C12, C13: 220u, rcl:CPOL-EU153CLV-0605
- added D7: (no value), dp_devices:DIODE-DO-214AC
- added IC1: (no value), linear:LM2596S
- added L1: (no value), SparkFun-Passives:INDUCTORPWR
- added U$5: CQ-121, Mantech.co.za:CQ-121
Connections:
- new net N$1: D7.C, IC1.OUT, L1.1
- net +12V: now also C13.+, IC1.FB, L1.2
- net +24V: now also C12.+, IC1.IN, U$5.2; no longer F2.2
- net GND: now also C12.-, C13.-, D7.A, IC1.EN, IC1.GND, IC1.GND@1
- net PWRIN: now also U$5.1; no longer F2.1
Other:
- note added: "RAMPS 1.5 Google Plus Edition (RepRap Arduino Mega Pololu Shield) Development started by Peter van der Walt and ThantiK on 5 Oc\t 2014"
- note removed: "RAMPS 1.5 Google Plus Edition (RepRap Arduino Mega Pololu Shield) Development started by Peter van der Walt and ThantiK on 5 OCt 2014"
Changed lines of the file:
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@@
 </variantdefs>
 <classes>
-<class number="0" name="default" width="0" drill="0">
+<class number="0" name="default" width="0.254" drill="0">
+<clearance class="0" value="0.254"/>
 </class>
 </classes>
@@
 <part name="C7" library="SparkFun-Capacitors" deviceset="CAP_POL" device="D" value="100U"/>
 <part name="C9" library="SparkFun-Capacitors" deviceset="CAP_POL" device="D" value="100U"/>
-<part name="F2" library="fuse" deviceset="FUSE" device="GSH15"/>
 <part name="R2" library="adafruit" deviceset="R-US_" device="M1206" value="1K"/>
 <part name="DEADFUSE" library="led" deviceset="LED" device="CHIPLED_1206"/>
@@
 <part name="SJ15" library="jumper" deviceset="SJ" device=""/>
 <part name="U$4" library="Communica.co.za" deviceset="XY825A-8P" device=""/>
+<part name="U$5" library="Mantech.co.za" deviceset="CQ-121" device=""/>
+<part name="IC1" library="linear" deviceset="LM2596S" device=""/>
+<part name="L1" library="SparkFun-Passives" deviceset="INDUCTOR" device="PWR"/>
+<part name="D7" library="dp_devices" deviceset="DIODE" device="-DO-214AC"/>
+<part name="C12" library="rcl" deviceset="CPOL-EU" device="153CLV-0605" value="220u"/>
+<part name="C13" library="rcl" deviceset="CPOL-EU" device="153CLV-0605" value="220u"/>
 </parts>
 <sheets>
@@
 <text x="165.1" y="96.52" size="5.08" layer="108">GPL v3</text>
 <text x="-17.78" y="111.76" size="3.81" layer="108">RAMPS 1.5 Google Plus Edition (RepRap Arduino Mega Pololu Shield)
-Development started by Peter van der Walt and ThantiK on 5 OCt 2014</text>
+Development started by Peter van der Walt and ThantiK on 5 Oc\t 2014</text>
 <text x="195.58" y="96.52" size="1.778" layer="108">UltiMachine</text>
 <text x="-17.78" y="99.06" size="6.4516" layer="108">reprap.org/wiki/RAMPS</text>
@@
 <text x="-15.24" y="58.42" size="1.778" layer="95">PWR For Atmega from 12v rail</text>
 <wire x1="-20.32" y1="-22.86" x2="7.62" y2="-22.86" width="0.1524" layer="95"/>
-<wire x1="7.62" y1="-22.86" x2="7.62" y2="27.94" width="0.1524" layer="95"/>
 <wire x1="96.52" y1="-71.12" x2="99.06" y2="-71.12" width="0.1524" layer="95"/>
 <wire x1="99.06" y1="-71.12" x2="99.06" y2="27.94" width="0.1524" layer="95"/>
@@
 <instance part="C7" gate="G$1" x="203.2" y="-5.08" rot="R270"/>
 <instance part="C9" gate="G$1" x="233.68" y="-5.08" rot="R270"/>
-<instance part="F2" gate="G$1" x="-58.42" y="-25.4"/>
 <instance part="R2" gate="G$1" x="-58.42" y="-20.32" rot="R180"/>
 <instance part="DEADFUSE" gate="G$1" x="-48.26" y="-20.32" rot="R90"/>
@@
 <instance part="SJ15" gate="1" x="238.76" y="-50.8" rot="R90"/>
 <instance part="U$4" gate="G$1" x="86.36" y="-68.58" rot="R90"/>
+<instance part="U$5" gate="G$1" x="-60.96" y="-25.4"/>
+<instance part="IC1" gate="G$1" x="-68.58" y="-116.84"/>
+<instance part="L1" gate="G$1" x="-48.26" y="-114.3" rot="R90"/>
+<instance part="D7" gate="D" x="-55.88" y="-119.38" rot="R90"/>
+<instance part="C12" gate="G$1" x="-81.28" y="-116.84"/>
+<instance part="C13" gate="G$1" x="-40.64" y="-116.84"/>
 </instances>
 <busses>
@@
 <label x="66.04" y="-66.04" size="1.778" layer="95"/>
 </segment>
+<segment>
+<pinref part="IC1" gate="G$1" pin="EN"/>
+<pinref part="IC1" gate="G$1" pin="GND"/>
+<wire x1="-78.74" y1="-121.92" x2="-78.74" y2="-129.54" width="0.1524" layer="91"/>
+<wire x1="-78.74" y1="-129.54" x2="-68.58" y2="-129.54" width="0.1524" layer="91"/>
+<wire x1="-68.58" y1="-129.54" x2="-68.58" y2="-127" width="0.1524" layer="91"/>
+<wire x1="-68.58" y1="-129.54" x2="-66.04" y2="-129.54" width="0.1524" layer="91"/>
+<pinref part="IC1" gate="G$1" pin="GND@1"/>
+<wire x1="-66.04" y1="-129.54" x2="-66.04" y2="-127" width="0.1524" layer="91"/>
+<junction x="-68.58" y="-129.54"/>
+<wire x1="-78.74" y1="-119.38" x2="-78.74" y2="-121.92" width="0.1524" layer="91"/>
+<label x="-86.36" y="-124.46" size="1.778" layer="95"/>
+<pinref part="D7" gate="D" pin="A"/>
+<wire x1="-55.88" y1="-121.92" x2="-55.88" y2="-129.54" width="0.1524" layer="91"/>
+<wire x1="-55.88" y1="-129.54" x2="-66.04" y2="-129.54" width="0.1524" layer="91"/>
+<junction x="-66.04" y="-129.54"/>
+<wire x1="-78.74" y1="-121.92" x2="-81.28" y2="-121.92" width="0.1524" layer="91"/>
+<wire x1="-81.28" y1="-121.92" x2="-81.28" y2="-124.46" width="0.1524" layer="91"/>
+<wire x1="-55.88" y1="-129.54" x2="-40.64" y2="-129.54" width="0.1524" layer="91"/>
+<wire x1="-55.88" y1="-129.54" x2="-38.1" y2="-129.54" width="0.1524" layer="91"/>
+<label x="-38.1" y="-129.54" size="1.778" layer="95"/>
+<junction x="-78.74" y="-121.92"/>
+<junction x="-78.74" y="-119.38"/>
+<junction x="-55.88" y="-121.92"/>
+<junction x="-55.88" y="-129.54"/>
+<pinref part="C12" gate="G$1" pin="-"/>
+<junction x="-81.28" y="-121.92"/>
+<pinref part="C13" gate="G$1" pin="-"/>
+<wire x1="-40.64" y1="-121.92" x2="-40.64" y2="-129.54" width="0.1524" layer="91"/>
+</segment>
 </net>
 <net name="VCC" class="0">
@@
 <wire x1="-7.62" y1="-99.06" x2="-7.62" y2="-96.52" width="0.1524" layer="91"/>
 </segment>
+<segment>
+<pinref part="L1" gate="G$1" pin="2"/>
+<label x="-40.64" y="-109.22" size="1.778" layer="95"/>
+<junction x="-40.64" y="-114.3"/>
+<pinref part="IC1" gate="G$1" pin="FB"/>
+<wire x1="-58.42" y1="-119.38" x2="-58.42" y2="-116.84" width="0.1524" layer="91"/>
+<wire x1="-58.42" y1="-116.84" x2="-63.5" y2="-116.84" width="0.1524" layer="91"/>
+<wire x1="-63.5" y1="-116.84" x2="-63.5" y2="-109.22" width="0.1524" layer="91"/>
+<wire x1="-63.5" y1="-109.22" x2="-40.64" y2="-109.22" width="0.1524" layer="91"/>
+<wire x1="-40.64" y1="-109.22" x2="-40.64" y2="-114.3" width="0.1524" layer="91"/>
+<pinref part="C13" gate="G$1" pin="+"/>
+<junction x="-40.64" y="-114.3"/>
+</segment>
 </net>
 <net name="E0-STEP" class="0">
@@
 <net name="PWRIN" class="0">
 <segment>
-<wire x1="-68.58" y1="-25.4" x2="-63.5" y2="-25.4" width="0.1524" layer="91"/>
-<pinref part="F2" gate="G$1" pin="1"/>
+<wire x1="-68.58" y1="-25.4" x2="-66.04" y2="-25.4" width="0.1524" layer="91"/>
 <pinref part="R2" gate="G$1" pin="2"/>
+<wire x1="-66.04" y1="-25.4" x2="-63.5" y2="-25.4" width="0.1524" layer="91"/>
 <wire x1="-63.5" y1="-20.32" x2="-68.58" y2="-20.32" width="0.1524" layer="91"/>
 <wire x1="-68.58" y1="-20.32" x2="-68.58" y2="-25.4" width="0.1524" layer="91"/>
@@
 <pinref part="PWRIN" gate="-1" pin="KL"/>
 <label x="-76.2" y="-20.32" size="1.778" layer="95"/>
+<pinref part="U$5" gate="G$1" pin="1"/>
+<junction x="-66.04" y="-25.4"/>
 </segment>
 <segment>
@@
 </segment>
 <segment>
-<wire x1="-53.34" y1="-25.4" x2="-43.18" y2="-25.4" width="0.1524" layer="91"/>
+<wire x1="-53.34" y1="-25.4" x2="-50.8" y2="-25.4" width="0.1524" layer="91"/>
+<wire x1="-50.8" y1="-25.4" x2="-43.18" y2="-25.4" width="0.1524" layer="91"/>
 <wire x1="-43.18" y1="-27.94" x2="-43.18" y2="-25.4" width="0.1524" layer="91"/>
 <junction x="-43.18" y="-25.4"/>
 <pinref part="D2" gate="G$1" pin="C"/>
-<pinref part="F2" gate="G$1" pin="2"/>
 <pinref part="DEADFUSE" gate="G$1" pin="C"/>
 <wire x1="-43.18" y1="-25.4" x2="-43.18" y2="-20.32" width="0.1524" layer="91"/>
 <label x="-40.64" y="-25.4" size="1.778" layer="95"/>
 <wire x1="-43.18" y1="-25.4" x2="-33.02" y2="-25.4" width="0.1524" layer="91"/>
+<pinref part="U$5" gate="G$1" pin="2"/>
+<junction x="-50.8" y="-25.4"/>
 </segment>
 <segment>
@@
 <label x="66.04" y="-48.26" size="1.778" layer="95"/>
 </segment>
+<segment>
+<pinref part="IC1" gate="G$1" pin="IN"/>
+<wire x1="-78.74" y1="-114.3" x2="-81.28" y2="-114.3" width="0.1524" layer="91"/>
+<label x="-86.36" y="-111.76" size="1.778" layer="95"/>
+<wire x1="-81.28" y1="-114.3" x2="-81.28" y2="-111.76" width="0.1524" layer="91"/>
+<junction x="-78.74" y="-114.3"/>
+<pinref part="C12" gate="G$1" pin="+"/>
+<junction x="-81.28" y="-114.3"/>
+</segment>
 </net>
 <net name="12V" class="0">
@@
 </segment>
 </net>
+<net name="N$1" class="0">
+<segment>
+<pinref part="IC1" gate="G$1" pin="OUT"/>
+<wire x1="-58.42" y1="-114.3" x2="-55.88" y2="-114.3" width="0.1524" layer="91"/>
+<pinref part="D7" gate="D" pin="C"/>
+<wire x1="-55.88" y1="-114.3" x2="-55.88" y2="-116.84" width="0.1524" layer="91"/>
+<pinref part="L1" gate="G$1" pin="1"/>
+<junction x="-55.88" y="-114.3"/>
+<junction x="-58.42" y="-114.3"/>
+</segment>
+</net>
